File: FPGA_Power.kicad_sch (KiCad schematic)
At the start: 13 parts, among them U5 NCP115AMX120TCG, U9 ICE40UP5K-SG48ITR

Commit message: Working on the schematic
Parts:
- removed SJ6: SHORT, Jumper:SolderJumper-2_P1.3mm_Bridged_RoundedPad1.0x1.5mm, symbol UPduino_v3.0:Device_R
- added JP1: Jumper_2_Bridged, symbol Jumper:Jumper_2_Bridged
Connections:
- net +1.2V_CORE: now also JP1.2 (B)
- net +1V2: now also JP1.1 (A)
- net +3V3_FPGA renamed +3V3
Other:
- note removed: "Core current measurement"
