File: DDC_SDR.kicad_sch (KiCad schematic)
At the start: 23 parts, among them Q3 2N7002, U2 MS9280, U3 AD9708AR, U7 ICE40UP5K-SG48ITR, U8 W25Q32JVSSIQ

Commit message: Working on the schematic
Parts:
- removed JP67: Jumper_2_Bridged, Jumper:SolderJumper-2_P1.3mm_Bridged2Bar_RoundedPad1.0x1.5mm, symbol Jumper:Jumper_2_Bridged
- removed SJ3: SHORT, Jumper:SolderJumper-2_P1.3mm_Bridged_RoundedPad1.0x1.5mm, symbol UPduino_v3.0:Device_R
- added C15: 1uF, PCM_JLCPCB:C_0805, symbol PCM_JLCPCB-Capacitors:0805,1uF
- added C23, C34, C93: 100nF, PCM_JLCPCB:C_0805, symbol PCM_JLCPCB-Capacitors:0805,100nF
- added C44: 10uF, PCM_JLCPCB:C_1206, symbol PCM_JLCPCB-Capacitors:1206,10uF
- added C51, C64, C65, C66: 0.1u, Capacitor_SMD:C_0402_1005Metric, symbol UPduino_v3.0:Device_C
- added C84, C91: 100uF, PCM_JLCPCB:C_CASE-B-3528-21(mm), symbol PCM_JLCPCB-Capacitors:CASE-B-3528-21(mm),100uF
- added JP50: USB_ONLY, Jumper:SolderJumper-2_P1.3mm_Bridged2Bar_RoundedPad1.0x1.5mm, symbol Jumper:Jumper_2_Bridged
- added R15, R16: 10kΩ, PCM_JLCPCB:R_0805, symbol PCM_JLCPCB-Resistors:0805,10kΩ
- added TP13: VA/2, TP_Label:TestPoint_THTPad_D2.0mm_Drill1.0mm, symbol Connector:TestPoint
- A2: value RaspberryPi_Pico_W -> RaspberryPi_or_Pico_W_2_or_2W_or_YD-RP2040
Connections:
- net VIO_BANK_2 is gone; now on net +3V3: C30.1, C32.1, U7.1 (VCCIO_2)
- net +3V3: now also C21.1, C22.1, C38.1, C39.1, U2.2 (DRVDD), U3.27 (DVDD), U7.22 (SPI_VCCIO1), U7.33 (VCCIO_0)
- net +3V3_FPGA: no longer C21.1, C22.1, C38.1, C39.1, U2.23 (MODE), U7.22 (SPI_VCCIO1), U7.33 (VCCIO_0)
- net ADC_CLK: now also U2.15 (CLK)
- net D0: now also U2.5 (D0)
- net D1: now also U2.6 (D1)
- net D2: now also U2.7 (D2)
- net D3: now also U2.8 (D3)
- net D4: now also U2.9 (D4)
- net D5: now also U2.10 (D5)
- net D6: now also U2.11 (D6)
- net D7: now also U2.12 (D7)
- net GND: now also U2.1 (AVSS), U2.14 (DRVSS), U2.18 (REFSENSE), C15.2, C64.2, C65.2, C66.2
- net ICE_DONE: now also U7.7 (CDONE)
- net at U2.21 (REFTS): now also TR2.6 (RD+), U2.25 (REFBS)
- net at U2.22 (REFTF): now also C44.1, C51.1, C65.1
- net at U2.24 (REFBF): now also C44.2, C51.2, C64.1
- net at U2.26 (VREF): now also C15.1, C66.1
- net at U2.27 (AIN): now also TR2.8 (RD-)
- net VDDA: now reaches U2.28 (AVDD)
- net VDDA: now also C34.2, C84.1, C93.2, R15.2
- net at A2.39 (VSYS): now also JP50.2 (B)
- net +4.7V: now reaches A2.40 (VBUS)
- net +4.7V: now also JP50.1 (A)
- net VA/2: now reaches TR2.7 (C_RD)
- net VA/2: now also U2.23 (MODE), C23.2, C84.2, C91.1, C93.1, R15.1, R16.2, TP13.1
- new net GNDA: C23.1, C34.1, C91.2, R16.1
Other:
- note added: "For the YD-RP2040 we want the USB Only jumper shorted."
- note added: "If you are using a real Pico, this jumper bridges a Schottky diode from USB in to Vsys (4.7v with it open, 5.0v from USB port with it soldered)"
- note removed: "Bank 1 is 3.3V IO!"
- note removed: "DAC Data Bus (8 Pins): Pins 48, 47, 46, 45, 44, 4, 3, 2. (This routes the transmitting DAC entirely to the bottom edge of the board, isolating it from the ADC). DAC Clock OUT: Pin 6 (This is IOB_13b on Bank 1, which sits physically right next to the Bank 2 pins on the right side of the chip)."
- note removed: "I2S Bus (BCLK, LRCLK, RX, TX): Pins 18, 19, 20, 21 (Pin 20 is a GBIN, which is great if the Pico ever needs to send a master clock)."
- note removed: "Note: Output-only when the pll is used for 2 output mode"
- note removed: "Top Edge (Near the corner): Pin 37 (G1): 30.72 MHz Clock IN (From Oscillator) Right Edge (Going down the side of the chip): Pin 36: Spare (Perfect for a test point or interrupt) Pin 35 (G0): ADC Clock OUT Pin 34: ADC_D7 (MSB) Pin 33: (VCCIO_0 - Power Via) Pin 32: ADC_D6 Pin 31: ADC_D5 Pin 30: (VCC - Power Via) Pin 29: (VCCPLL - Power Via) Pin 28: ADC_D4 Pin 27: ADC_D3 Pin 26: ADC_D2 Pin 25: ADC_D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"
- moved on the sheet: C21, C22, C30, C32, C38, C39, R14, TR2, U7A, U7B, U7C

Commit message: Much Schematic Progress
Parts:
- removed C21, C32, C39, C51, C64, C65, C66: 0.1u, Capacitor_SMD:C_0402_1005Metric, symbol UPduino_v3.0:Device_C
- removed C22, C30, C38: 4.7u, Capacitor_SMD:C_0402_1005Metric, symbol UPduino_v3.0:Device_C
- removed R11: 22, Resistor_SMD:R_0402_1005Metric, symbol Device:R
- removed R13, R14, R23: 10K, Resistor_SMD:R_0402_1005Metric, symbol Device:R
- removed R8: 10K, Resistor_SMD:R_0402_1005Metric, symbol UPduino_v3.0:Device_R
- removed RN1: 10K, Resistor_SMD:R_Array_Concave_4x0402, symbol Device:R_Pack04_Split
- added C100, C101, C102, C16, C18, C19, C20, C21, C22, C28, C29, C31, C32, C38, C52, C66, C67, C7, C97, C98, C99: 100nF, PCM_JLCPCB:C_0402, symbol PCM_JLCPCB-Capacitors:0402,100nF,(2)
- added C30: 100nF, PCM_JLCPCB:C_0805, symbol PCM_JLCPCB-Capacitors:0805,100nF
- added C63, C64, C65: 4.7uF, PCM_JLCPCB:C_0402, symbol PCM_JLCPCB-Capacitors:0402,4.7uF
- added D6: Green, PCM_JLCPCB:D_0805, symbol PCM_JLCPCB-Diodes:LED,0805,Green
- added D7: Red, PCM_JLCPCB:D_0805, symbol PCM_JLCPCB-Diodes:LED,0805,Red
- added D8: Yellow, PCM_JLCPCB:D_0805, symbol PCM_JLCPCB-Diodes:LED,0805,Yellow
- added J13: AWG_OUT, Intro_to_CAD:Conn_Coaxial_Frohne, symbol Connector:Conn_Coaxial
- added J14: DUT, Intro_to_CAD:Conn_Coaxial_Frohne, symbol Connector:Conn_Coaxial
- added J3, J4: Filter, symbol Connector:Conn_01x04_Socket
- added J6: PMOD, symbol Connector_Generic:Conn_01x06
- added Q10: 2N7002, PCM_JLCPCB:Q_SOT-23, symbol JLCPCB-Transistors:NMOS,2N7002
- added R11: 22Ω, PCM_JLCPCB:R_0402, symbol PCM_JLCPCB-Resistors:0402,22Ω
- added R13, R14, R18, R23, R26, R27, R29, R64, R67, R68, R69, R8: 10kΩ, PCM_JLCPCB:R_0402, symbol PCM_JLCPCB-Resistors:0402,10kΩ
- added R17, R62, R63, R65, R66, R9: 49.9Ω, PCM_JLCPCB:R_0402, symbol PCM_JLCPCB-Resistors:0402,49.9Ω
- added R30, R35: 10kΩ, PCM_JLCPCB:R_0805, symbol PCM_JLCPCB-Resistors:0805,10kΩ
- added R36, R60: 100Ω, PCM_JLCPCB:R_0805, symbol PCM_JLCPCB-Resistors:0805,100Ω
- added R37, R61: 300Ω, PCM_JLCPCB:R_0805, symbol PCM_JLCPCB-Resistors:0805,300Ω
- added R4: 2kΩ, PCM_JLCPCB:R_0805, symbol PCM_JLCPCB-Resistors:0805,2kΩ
- added R70, R71, R72: 330Ω, PCM_JLCPCB:R_0402, symbol PCM_JLCPCB-Resistors:0402,330Ω
- added S1: Tactile Button, 160gf, PCM_JLCPCB:SW_TS-1088-AR02016, symbol PCM_JLCPCB-Connectors_Buttons:Tactile Button, 160gf, 12V, 50mA, 4.0mm
- added TR3, TR4: H1102NLT, Intro_to_CAD:XFMR_H1102NLT, symbol Transformer:PT61017PEL
- added U15, U25: TPH2501-TR, Package_TO_SOT_SMD:SOT-23-5, symbol Amplifier_Operational:TLV3541xDBV
- added U26: 74LVC1G3157GW, symbol 74xGxx:74LVC1G3157
- U3: LCSC (none) -> C1509022
Connections:
- net +3V3: now also D4.2 (A), C102.1, C16.1, C18.1, C32.1, C38.1, C63.1, C64.1, C65.1, J6.6 (Pin_6), R13.1, R23.1, R69.1
- net +3V3_FPGA: now also R8.1; no longer D4.2 (A)
- net BCK: now also U7.11 (IOB_20a)
- net GND: now also TR2.11 (RX+), U3.15 (SLEEP), U3.16 (REFLO), U3.20 (ACOM), U3.26 (DCOM), C100.2, C101.2, C102.2, C16.2, C18.2, C19.2, C21.2, C22.2, C28.2, C31.2, C32.2, C38.2, C52.2, C63.2, C64.2, C65.2, C66.2, C67.2, C97.2, J13.2 (Ext), J14.2 (Ext), J3.2 (Pin_2), J3.3 (Pin_3), J4.2 (Pin_2), J4.3 (Pin_3), J6.5 (Pin_5), Q10.2 (S), R14.2, R17.2, R18.2, R26.2, R27.2, R29.2, R4.2, R60.1, R63.2, R64.2, R9.2, S1.1 (A), TR3.14 (TX-), TR4.6 (RD+), U15.2 (V-), U25.2 (V-), U26.2 (GND)
- net GNDA: now also R35.1
- net ICE_12|IO2: now also R27.1
- net ICE_13|IO3: now also R29.1
- net ICE_SCK: now also R11.1, R18.1
- net ICE_SI: now also R26.1
- net ICE_SSN: now also R8.2
- net RX_DATA: now also U7.10 (IOB_18a)
- net SCL_GPIO3: now also R13.2
- net SDA_GPIO2: now also R23.2
- net TX_DATA: now also U7.9 (IOB_16a)
- net VDDA: now also U3.24 (AVDD), C101.1, C20.1, C22.1, C52.1, C67.1, C97.1, R30.2, R67.1, R68.1, U15.5 (V+), U25.5 (V+), U26.5 (VCC)
- net WS: now also U7.18 (IOB_31b)
- net ~{ICE_RST}: now also R14.1
- net at A2.9 (GPIO6): now also R11.2
- net at C44.1, U2.22 (REFTF): now also C29.1, C31.1
- net at C44.2, U2.24 (REFBF): now also C28.1, C29.2
- net at C15.1, U2.26 (VREF): now also C21.1
- net ~{T}/R: now reaches A2.31 (GPIO26_ADC0)
- net REF: now reaches A2.32 (GPIO27_ADC1)
- net REF: now also Q10.1 (G)
- net at TR2.9 (RX-): now also C99.2
- net PMOD_0: now reaches U7.19 (IOB_29b)
- net PMOD_0: now also J6.1 (Pin_1)
- net PMOD_1: now reaches U7.20 (IOB_25b_G3)
- net PMOD_1: now also J6.2 (Pin_2)
- net at U3.17 (REFIO): now also C19.1
- net at U3.18 (FS_ADJ): now also R4.1
- net at U3.19 (COMP1): now also C20.2
- net OB: now reaches U3.21 (IOUTB)
- net OB: now also R9.1, TR3.1 (TD+)
- net OA: now reaches U3.22 (IOUTA)
- net OA: now also R17.1, TR3.3 (TD-), U25.3 (+)
- net at U3.23 (COMP2): now also C100.1
- net PMOD_2: now reaches U7.38 (IOT_50b)
- net PMOD_2: now also J6.3 (Pin_3)
- net RED: now reaches U7.39 (RGB0)
- net RED: now also D7.1
- net YELLOW: now reaches U7.40 (RGB1)
- net YELLOW: now also D8.1
- net GREEN: now reaches U7.41 (RGB2)
- net GREEN: now also D6.1
- net FIL renamed BAND_SW
- net ICE42: no longer names the net of A2.26 (GPIO20)
- net ICE42: no longer U7.42 (IOT_51a)
- net ICE43 renamed FPGA_INT
- new net: R60.2, R61.1, U25.4 (-)
- new net: C30.1, TR3.16 (TX+)
- new net: R36.2, R37.1, U15.4 (-)
- new net: J4.1 (Pin_1), R37.2, U15.1
- new net: C30.2, J3.1 (Pin_1)
- new net: J3.4 (Pin_4), R30.1, R35.2, U15.3 (+)
- new net: R63.1, R65.1, TR4.9 (RX-)
- new net: C98.1, U26.3
- new net: C99.1, R64.1, R67.2, U26.4
- new net: J14.1 (In), R66.1, TR4.11 (RX+)
- new net: C98.2, TR4.8 (RD-)
- new net: J13.1 (In), R62.2
- new net: R61.2, R62.1, U25.1
- new net: C66.1, R36.1
- new net: D6.2, R72.2
- new net: D8.2, R70.2
- new net: D7.2, R71.2
- new net PMOD0: R69.2, S1.2 (B)
- new net PMOD_3: J6.4 (Pin_4), U7.42 (IOT_51a)
- new net RX_OUT: U26.1
- new net TX_OUT: C7.1, J4.4 (Pin_4)
- new net VNA_RF: R65.2, R66.2
- new net ~{REF}: Q10.3 (D), R68.2, U26.6
- no-connect marks 3 -> 24
Other:
- sheet Filter Playground ports: added BAND_SW, RX_OUT, TX_OUT, ~{T}/R; removed none
- sheet Programmable Gain Amplifier ports: added PGA0, PGA1, PGA2, PGA3, PGA_IN, PGA_OUT; removed none
- note added: "DAC Outputs"
- note added: "Reflection Bridge"
- note added: "Traffic Lights"
- moved on the sheet: C23, C27, C34, C84, C91, C93, D4, Q3, R15, R16, U8

Commit message: Fixing lots of schematic issues
Parts:
- removed R30, R35: 10kΩ, PCM_JLCPCB:R_0805, symbol PCM_JLCPCB-Resistors:0805,10kΩ
- removed R64, R67: 10kΩ, PCM_JLCPCB:R_0402, symbol PCM_JLCPCB-Resistors:0402,10kΩ
- added C103, C8, C9: 100nF, PCM_JLCPCB:C_0402, symbol PCM_JLCPCB-Capacitors:0402,100nF,(2)
- added JP4: Jumper_2_Open, Jumper:SolderJumper-2_P1.3mm_Open_RoundedPad1.0x1.5mm, symbol Jumper:Jumper_2_Open
- added JP51: ICE20_G3, Jumper:SolderJumper-2_P1.3mm_Bridged2Bar_RoundedPad1.0x1.5mm, symbol Jumper:Jumper_2_Bridged
- added R76, R79: 10kΩ, PCM_JLCPCB:R_0402, symbol PCM_JLCPCB-Resistors:0402,10kΩ
- U26: footprint (none) -> PCM_JLCPCB:SOT-363_SC-70-6
Connections:
- net SCL_GPIO3 is gone; now on net SCL: A2.5 (GPIO3), R13.2
- net SDA_GPIO2 is gone; now on net SDA: A2.4 (GPIO2), R23.2
- net VNA_RF is gone; now on net TX_OUT: R65.2, R66.2
- net +3V3: now also R70.1, R71.1, R72.1
- net AF_DAC_DATA: now also A2.22 (GPIO17); no longer A2.1 (GPIO0)
- net AF_DAC_LRCK: now also A2.26 (GPIO20); no longer A2.24 (GPIO18)
- net AF_DAC_MCLK: now also A2.24 (GPIO18); no longer A2.2 (GPIO1)
- net AF_DAC_SCLK: now also A2.25 (GPIO19); no longer A2.22 (GPIO17)
- net FPGA_INT: now also A2.1 (GPIO0); no longer A2.25 (GPIO19)
- net PMOD0: now also JP4.1 (A); no longer R69.2, S1.2 (B)
- net PMOD_1: now also U7.42 (IOT_51a); no longer U7.20 (IOB_25b_G3)
- net PMOD_3: now also U7.20 (IOB_25b_G3), JP51.1 (A); no longer U7.42 (IOT_51a)
- net RX_OUT: now also C103.1; no longer U26.1
- net TX_OUT: now also C7.2; no longer C7.1, J4.4 (Pin_4)
- net VA/2: now also R76.1, R79.1
- net WS: now also U7.21 (IOB_23b); no longer U7.18 (IOB_31b)
- net at R37.2, U15.1: now also C8.1; no longer J4.1 (Pin_1)
- net at J3.4 (Pin_4): now also C9.1; no longer U15.3 (+)
- net at A2.34 (GPIO28_ADC2): now also JP51.2 (B)
- net at C99.1, U26.4: now also R76.2
- new net: C7.1, J4.4 (Pin_4)
- new net: C9.2, R79.2, U15.3 (+)
- new net: C103.2, U26.1
- new net: JP4.2 (B), R69.2, S1.2 (B)
- new net: C8.2, J4.1 (Pin_1)
- new net SPI_RUN_CS: A2.2 (GPIO1), U7.18 (IOB_31b)
Other:
- note added: "Note: When using the SPI during runtime, your Verilog must use the pin labelled ICE_SI as MISO, not MOSI. The Pico is the Master in runtime. This looks backwards, but the labeling had to be this way to be correct for the FPGA Flash."
- note added: "PMOD"
- note added: "The Arbitrary Waveform Generator puts out only positive voltages. 128 corresponds to: (10mA*50)*4 = 2 V 255 corresponds to: (20mA*50)*4 = 4 V 0 corresponds to: (0mA*50)*4 = 0"
- note removed: "Note: Bank 2 is selectable IO voltage! To select non-3.3V, cut the shorted jumper and supply external voltage (1.8-3.3V) on VIO_BANK_2."
- moved on the sheet: C23, C27, C34, C52, C7, C84, C91, C93, C99, D6, D7, D8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

Commit message: More fixes
Parts:
- removed R37: 300Ω, PCM_JLCPCB:R_0805, symbol PCM_JLCPCB-Resistors:0805,300Ω
- added JP5, JP6, JP7: Jumper_2_Open, Jumper:SolderJumper-2_P1.3mm_Open_RoundedPad1.0x1.5mm, symbol Jumper:Jumper_2_Open
- added R37: 100Ω, PCM_JLCPCB:R_0805, symbol PCM_JLCPCB-Resistors:0805,100Ω
Connections:
- net PMOD_0: now also JP5.2 (B)
- net PMOD_1: now also JP6.2 (B)
- net PMOD_3: now also JP7.2 (B)
- net at R36.2, U15.4 (-): now also R37.1
- net at C8.1, U15.1: now also R37.2
- new net Angle Encoder/GPIO_A: JP5.1 (A)
- new net Angle Encoder/GPIO_B: JP6.1 (A)
- new net Angle Encoder/GPIO_C: JP7.1 (A)
Other:
- sheet Angle Encoder ports: added GPIO_A, GPIO_B, GPIO_C; removed none
- moved on the sheet: C66, R36

Commit message: Fixed a lot more mistakes...
Parts:
- removed D4: LTST-C191KGKT, LED_SMD:LED_0603_1608Metric, symbol UPduino_v3.0:Device_LED_ALT
- added C106, C107: 100nF, PCM_JLCPCB:C_0402, symbol PCM_JLCPCB-Capacitors:0402,100nF,(2)
- added D4: White, PCM_JLCPCB:D_0805, symbol PCM_JLCPCB-Diodes:LED,0805,White
- added J16: S12_OUT, Intro_to_CAD:Conn_Coaxial_Frohne, symbol Connector:Conn_Coaxial
- added R30: 22Ω, PCM_JLCPCB:R_0402, symbol PCM_JLCPCB-Resistors:0402,22Ω
- added R35: 49.9Ω, PCM_JLCPCB:R_0402, symbol PCM_JLCPCB-Resistors:0402,49.9Ω
- added R80: 330Ω, PCM_JLCPCB:R_0402, symbol PCM_JLCPCB-Resistors:0402,330Ω
- added R81: 10kΩ, PCM_JLCPCB:R_0402, symbol PCM_JLCPCB-Resistors:0402,10kΩ
- added TP29: U15, TestPoint:TestPoint_THTPad_D2.5mm_Drill1.2mm, symbol Connector:TestPoint
- added TP30: U25, TestPoint:TestPoint_THTPad_D2.5mm_Drill1.2mm, symbol Connector:TestPoint
- added U27: 74LVC1G3157GW, PCM_JLCPCB:SOT-363_SC-70-6, symbol 74xGxx:74LVC1G3157
- TP13: footprint TP_Label:TestPoint_THTPad_D2.0mm_Drill1.0mm -> TestPoint:TestPoint_THTPad_D2.5mm_Drill1.2mm
- TR4: Price (none) -> $0.21
- U2: LCSC (none) -> C1509022; Price (none) -> $1.52
- U25: Price (none) -> $0.35
- U26, U7: Price (none) -> $0.09
- U3: Price (none) -> $1.90
Connections:
- net +3V3_FPGA is gone; now on net +3V3: C27.1, R8.1, U8.8 (VCC)
- net +3V3: now also R80.1
- net GND: now also C106.2, U27.2 (GND)
- net RX_OUT: now also U26.1; no longer C103.1
- net TX_OUT: now also C103.2; no longer R65.2, R66.2
- net VA/2: now also R81.1
- net VDDA: now also C106.1, U27.5 (VCC)
- net ~{REF}: now also U27.6
- net at A2.34 (GPIO28_ADC2): now also R30.1; no longer JP51.2 (B)
- net at Q3.3 (D): now also D4.1
- net at R37.2, U15.1: now also R35.1, TP29.1; no longer C8.1
- net at J13.1 (In), R62.2: now also C107.2
- net at R61.2, R62.1, U25.1: now also TP30.1
- new net: C8.1, R35.2
- new net: C103.1, R81.2, U27.4
- new net: R65.2, R66.2
- new net: JP51.2 (B), R30.2
- new net: D4.2, R80.2
- new net: C107.1, J16.1 (In)
- new net TX_REFL: U27.3
- new net TX_SDR: U27.1
- no-connect marks 24 -> 25
Other:
- note added: "ADC"
- note added: "DAC"
- note added: "Pico"
- moved on the sheet: C7, C8, J4, Q3

Commit message: Switching TX for VNA too
Parts:
- added C108, C109: 100nF, PCM_JLCPCB:C_0402, symbol PCM_JLCPCB-Capacitors:0402,100nF,(2)
- J16: value S12_OUT -> S21_OUT
Connections:
- net TX_REFL: now also R65.2, R66.2, C109.1; no longer U27.3
- net TX_SDR: now also C108.1; no longer U27.1
- new net: C108.2, U27.1
- new net: C109.2, U27.3
Other:
- moved on the sheet: C103, R81, U27A

Commit message: Fixing more errors....
Parts:
- U3: value AD9708AR -> MS9708
Connections:
- net PMOD_2: now also JP7.2 (B)
- net PMOD_3: no longer JP7.2 (B)
Changed lines of the file:
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@@
 		)
 	)
-	(label "PMOD_3"
+	(label "PMOD_2"
 		(at 83.82 157.48 0)
 		(effects
@@
 			)
 		)
-		(property "Value" "AD9708AR"
+		(property "Value" "MS9708"
 			(at 395.8433 97.79 0)
 			(show_name no)

Commit message: Removed FPGA Flash
Parts:
- removed C27: 0.1u, Capacitor_SMD:C_0402_1005Metric, symbol UPduino_v3.0:Device_C
- removed JP5, JP6, JP7: Jumper_2_Open, Jumper:SolderJumper-2_P1.3mm_Open_RoundedPad1.0x1.5mm, symbol Jumper:Jumper_2_Open
- removed R26, R27, R29: 10kΩ, PCM_JLCPCB:R_0402, symbol PCM_JLCPCB-Resistors:0402,10kΩ
- removed U8: W25Q32JVSSIQ, Package_SO:SOIC-8_5.23x5.23mm_P1.27mm, symbol UPduino_v3.0:W25Q32JVSS-Memory_Flash
- added JP52: PMOD_2, Jumper:SolderJumper-2_P1.3mm_Bridged2Bar_RoundedPad1.0x1.5mm, symbol Jumper:Jumper_2_Bridged
- added R55: 22Ω, PCM_JLCPCB:R_0402, symbol PCM_JLCPCB-Resistors:0402,22Ω
- J6: now not fitted
- JP51: value ICE20_G3 -> GBIN_PMOD_3
Connections:
- net ICE_12|IO2 is gone; now on net WS: U7.12 (IOB_22a)
- net ICE_13|IO3 is gone; now on net FPGA_INT: U7.13 (IOB_24a)
- net +3V3: now also R8.2; no longer R8.1
- net ADC_CLK: now also R55.2; no longer U7.35 (IOT_46b_G0)
- net FPGA_INT: no longer U7.43 (IOT_49a)
- net ICE_SSN: now also R8.1; no longer R8.2
- net PMOD_0: now also U7.18 (IOB_31b); no longer U7.19 (IOB_29b)
- net PMOD_1: now also U7.19 (IOB_29b); no longer U7.42 (IOT_51a)
- net PMOD_2: now also U7.21 (IOB_23b), JP52.1 (A); no longer U7.38 (IOT_50b)
- net REF: now also A2.31 (GPIO26_ADC0); no longer A2.32 (GPIO27_ADC1)
- net WS: no longer U7.21 (IOB_23b)
- net ~{T}/R: now also A2.2 (GPIO1); no longer A2.31 (GPIO26_ADC0)
- net ICE_SCK renamed SPI0_CLK
- net ICE_SI renamed SPI0_RX
- net SPI0_RX: now also U7.14 (IOB_32a_SPI_SO); no longer U7.17 (IOB_33b_SPI_SI)
- net ICE_SO renamed SPI0_TX
- net SPI0_TX: now also U7.17 (IOB_33b_SPI_SI); no longer U7.14 (IOB_32a_SPI_SO)
- removed net SPI_RUN_CS: A2.2 (GPIO1), U7.18 (IOB_31b)
- new net: R55.1, U7.35 (IOT_46b_G0)
- new net: A2.32 (GPIO27_ADC1), JP52.2 (B)
- new net ANG_0: U7.38 (IOT_50b)
- new net ANG_1: U7.42 (IOT_51a)
- new net ANG_2: U7.43 (IOT_49a)
Other:
- note added: "Button"
- note removed: "FPGA Flash"
- note removed: "Note: When using the SPI during runtime, your Verilog must use the pin labelled ICE_SI as MISO, not MOSI. The Pico is the Master in runtime. This looks backwards, but the labeling had to be this way to be correct for the FPGA Flash."
- moved on the sheet: D6, D7, D8, JP4, R18, R69, R70, R71, R72, R8, S1
