File: PGA.kicad_sch (KiCad schematic)
At the start: 11 parts, among them U1 TPH2501-TR, U10 74LVC1G3157GW, U13 TPH2501-TR

Commit message: Working on the schematic
Parts:
- removed C20, C33, C81: 100nF, PCM_JLCPCB:C_0805, symbol PCM_JLCPCB-Capacitors:0805,100nF
- removed C82, C83: 100uF, PCM_JLCPCB:C_CASE-B-3528-21(mm), symbol PCM_JLCPCB-Capacitors:CASE-B-3528-21(mm),100uF
- removed R4, R9: 10kΩ, PCM_JLCPCB:R_0805, symbol PCM_JLCPCB-Resistors:0805,10kΩ
- removed TP11: VA/2, TP_Label:TestPoint_THTPad_D2.0mm_Drill1.0mm, symbol Connector:TestPoint
Other:
- moved on the sheet: U10B

Commit message: Much Schematic Progress
Parts:
- removed U1, U13: TPH2501-TR, Package_TO_SOT_SMD:SOT-23-5, symbol Amplifier_Operational:TLV3541xDBV
- added C69, C70, C71, C72, C73, C74, C78, C79, C80, C81, C82, C83, C94, C95, C96: 100nF, PCM_JLCPCB:C_0402, symbol PCM_JLCPCB-Capacitors:0402,100nF,(2)
- added Q6, Q7, Q8, Q9: 2N7002, PCM_JLCPCB:Q_SOT-23, symbol JLCPCB-Transistors:NMOS,2N7002
- added R38, R40: 49.9Ω, PCM_JLCPCB:R_0805, symbol PCM_JLCPCB-Resistors:0805,49.9Ω
- added R39, R41: 510Ω, PCM_JLCPCB:R_0805, symbol PCM_JLCPCB-Resistors:0805,510Ω
- added R44, R45, R46, R47: 10kΩ, PCM_JLCPCB:R_0402, symbol PCM_JLCPCB-Resistors:0402,10kΩ
- added R48: 82Ω, PCM_JLCPCB:R_0603, symbol PCM_JLCPCB-Resistors:0603,82Ω
- added R49, R52: 22Ω, PCM_JLCPCB:R_0603, symbol PCM_JLCPCB-Resistors:0603,22Ω
- added R50, R51, R59: 10Ω, PCM_JLCPCB:R_0603, symbol PCM_JLCPCB-Resistors:0603,10Ω
- added R53: 33Ω, PCM_JLCPCB:R_0805, symbol PCM_JLCPCB-Resistors:0805,33Ω
- added R54: 2.2Ω, PCM_JLCPCB:R_0603, symbol PCM_JLCPCB-Resistors:0603,2.2Ω
- added R55, R56, R57, R58: 75Ω, PCM_JLCPCB:R_0402, symbol PCM_JLCPCB-Resistors:0402,75Ω
- added U13, U19, U20, U21, U22, U23, U24: 74LVC1G3157GW, symbol 74xGxx:74LVC1G3157
- added U16, U17: TPH2501-TR, Package_TO_SOT_SMD:SOT-23-5, symbol Amplifier_Operational:TLV3541xDBV
Connections:
- net at U10.1: now also R51.2
- net at U10.3: now also U13.3
- net at U10.6: now also Q6.3 (D), R44.2, U13.6
- net GND: now reaches U10.2 (GND)
- net GND: now also C69.2, C72.2, C73.2, C74.2, C78.2, C79.2, C80.2, C81.2, C82.2, C83.2, C94.2, C95.2, C96.2, Q6.2 (S), Q7.2 (S), Q8.2 (S), Q9.2 (S), U13.2 (GND), U16.2 (V-), U17.2 (V-), U19.2 (GND), U20.2 (GND), U21.2 (GND), U22.2 (GND), U23.2 (GND), U24.2 (GND)
- net VDDA: now reaches U10.5 (VCC)
- net VDDA: now also C69.1, C72.1, C73.1, C74.1, C78.1, C79.1, C80.1, C81.1, C82.1, C83.1, R44.1, R45.1, R46.1, R47.1, U13.5 (VCC), U16.5 (V+), U17.5 (V+), U19.5 (VCC), U20.5 (VCC), U21.5 (VCC), U22.5 (VCC), U23.5 (VCC), U24.5 (VCC)
- new net: R48.1, R50.2, R51.1
- new net: R55.2, R56.2, R57.1, R58.1, R59.2
- new net: R57.2, R58.2, U24.1
- new net: R40.2, R41.1, U17.4 (-)
- new net: C70.1, U19.1
- new net: U19.3, U20.3
- new net: Q7.3 (D), R45.2, U19.6, U20.6
- new net: R49.1, U21.1
- new net: U21.3, U22.3
- new net: Q8.3 (D), R46.2, U21.6, U22.6
- new net: C95.1, R54.2
- new net: C96.1, R59.1
- new net: Q9.3 (D), R47.2, U23.6, U24.6
- new net: C71.2, R40.1
- new net: C94.1, R48.2
- new net: R39.2, U16.1, U20.1
- new net: R52.2, U22.1
- new net: R49.2, R52.1, R53.1
- new net: R53.2, R54.1
- new net: R38.2, R39.1, U16.4 (-)
- new net: C70.2, R38.1
- new net: R55.1, R56.1, U23.1
- new net: R50.1, U13.1
- new net: U23.3, U24.3
- new net: C71.1, U24.4
- new net PGA0: Q6.1 (G)
- new net PGA1: Q8.1 (G)
- new net PGA2: Q9.1 (G)
- new net PGA3: Q7.1 (G)
- new net PGA_IN: U19.4
- new net PGA_OUT: R41.2, U17.1
- new net VA/2: U16.3 (+), U17.3 (+)
Other:
- note added: "10 dB Attenuator"
- note added: "20 dB Attenuator"
- note added: "5 dB Attenuator"
- moved on the sheet: U10A, U10B

Commit message: Fixing lots of schematic issues
Parts:
- removed R55, R56, R57, R58: 75Ω, PCM_JLCPCB:R_0402, symbol PCM_JLCPCB-Resistors:0402,75Ω
- removed R59: 10Ω, PCM_JLCPCB:R_0603, symbol PCM_JLCPCB-Resistors:0603,10Ω
- added R74: 49.9Ω, PCM_JLCPCB:R_0805, symbol PCM_JLCPCB-Resistors:0805,49.9Ω
- added R75: 10kΩ, PCM_JLCPCB:R_0402, symbol PCM_JLCPCB-Resistors:0402,10kΩ
- U10, U13, U19, U20, U21, U22, U23, U24: footprint (none) -> PCM_JLCPCB:SOT-363_SC-70-6
Connections:
- net GND: no longer C96.2
- net PGA_IN: now also R75.2
- net PGA_OUT: now also C96.2; no longer R41.2, U17.1
- net VA/2: now also R75.1
- net at U24.1: now also R41.2, U17.1
- net at U21.4: now also U10.4
- net at C96.1: now also U24.4
- net at R39.2, U16.1: now also R74.2; no longer U20.1
- net at U20.4: now also U13.4
- net at U22.4: now also U23.4
- net at U23.1: now also C71.1
- new net: R74.1, U20.1
Other:
- note removed: "20 dB Attenuator"
- moved on the sheet: C71, C72, Q7, R40, R41, R45, U17

Commit message: Fixed a lot more mistakes...
Parts:
- added TP31: U16, TestPoint:TestPoint_THTPad_D2.5mm_Drill1.2mm, symbol Connector:TestPoint
- added TP32: U17, TestPoint:TestPoint_THTPad_D2.5mm_Drill1.2mm, symbol Connector:TestPoint
- U10, U13, U19, U20, U21, U22, U23, U24: Price (none) -> $0.09
Connections:
- net at R41.2, U17.1, U24.1: now also TP32.1
- net at R39.2, R74.2, U16.1: now also TP31.1

Commit message: Added provision for switch leakage current.
Parts:
- removed C96: 100nF, PCM_JLCPCB:C_0402, symbol PCM_JLCPCB-Capacitors:0402,100nF,(2)
- added R26, R27, R29, R56, R57, R58: 100kΩ, PCM_JLCPCB:R_0402, symbol PCM_JLCPCB-Resistors:0402,100kΩ
Connections:
- net PGA_OUT: now also U24.4
- net VA/2: now also R26.1, R27.1, R29.1, R56.1, R57.1, R58.1
- net at U19.3, U20.3: now also R26.2
- net at R49.1, U21.1: now also R57.2
- net at U21.3, U22.3: now also R29.2
- net at U10.3, U13.3: now also R27.2
- net at R50.1, U13.1: now also R58.2
- net at U23.3, U24.3: now also R56.2

Commit message: Starting to place components
Parts:
- R38, R40, R74: footprint PCM_JLCPCB:R_0805 -> PCM_JLCPCB:R_0402; symbol PCM_JLCPCB-Resistors:0805,49.9Ω -> PCM_JLCPCB-Resistors:0402,49.9Ω; LCSC C17720 -> C25120; Overload Voltage (Max) 150V -> 50V; Part 0805W8F499JT5E -> 0402WGF499JTCE; Power(Watts) 125mW -> 62.5mW; Price 0.005USD -> 0.004USD; Stock 207522 -> 464542
Changed lines of the file:
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@@
 		)
 		(property "Voltage Rated" "50V"
-			(at 64.008 104.648 0)
+			(at 58.928 104.9162 0)
 			(show_name no)
 			(do_not_autoplace no)
@@
 		)
 		(property "Voltage Rated" "50V"
-			(at 229.108 33.528 0)
+			(at 224.028 33.7962 0)
 			(show_name no)
 			(do_not_autoplace no)
@@
 		)
 		(property "Voltage Rated" "50V"
-			(at 46.228 27.178 0)
+			(at 41.148 27.4462 0)
 			(show_name no)
 			(do_not_autoplace no)
@@
 		)
 		(property "Voltage Rated" "50V"
-			(at 122.428 109.728 0)
+			(at 117.348 109.9962 0)
 			(show_name no)
 			(do_not_autoplace no)
@@
 		)
 		(property "Voltage Rated" "50V"
-			(at 173.228 53.848 0)
+			(at 168.148 54.1162 0)
 			(show_name no)
 			(do_not_autoplace no)
@@
 		)
 		(property "Voltage Rated" "50V"
-			(at 216.408 118.618 0)
+			(at 211.328 118.8862 0)
 			(show_name no)
 			(do_not_autoplace no)
@@
 		)
 		(property "Voltage Rated" "50V"
-			(at 157.988 113.538 0)
+			(at 152.908 113.8062 0)
 			(show_name no)
 			(do_not_autoplace no)
@@
 		)
 		(property "Voltage Rated" "50V"
-			(at 243.078 118.618 0)
+			(at 237.998 118.8862 0)
 			(show_name no)
 			(do_not_autoplace no)
@@
 	)
 	(symbol
-		(lib_id "PCM_JLCPCB-Resistors:0805,49.9Ω")
+		(lib_id "PCM_JLCPCB-Resistors:0402,49.9Ω")
 		(at 217.17 48.26 90)
 		(unit 1)
@@
 			)
 		)
-		(property "Footprint" "PCM_JLCPCB:R_0805"
+		(property "Footprint" "PCM_JLCPCB:R_0402"
 			(at 217.17 50.038 90)
 			(hide yes)
@@
 			)
 		)
-		(property "Datasheet" "https://www.lcsc.com/datasheet/lcsc_datasheet_2206010200_UNI-ROYAL-Uniroyal-Elec-0805W8F499JT5E_C17720.pdf"
+		(property "Datasheet" "https://www.lcsc.com/datasheet/lcsc_datasheet_2205311900_UNI-ROYAL-Uniroyal-Elec-0402WGF499JTCE_C25120.pdf"
 			(at 217.17 48.26 0)
 			(hide yes)
@@
 			)
 		)
-		(property "Description" "125mW Thick Film Resistors 150V ±100ppm/°C ±1% 49.9Ω 0805 Chip Resistor - Surface Mount ROHS"
+		(property "Description" "62.5mW Thick Film Resistors 50V ±100ppm/°C ±1% 49.9Ω 0402 Chip Resistor - Surface Mount ROHS"
 			(at 217.17 48.26 0)
 			(hide yes)
@@
 			)
 		)
-		(property "LCSC" "C17720"
+		(property "LCSC" "C25120"
 			(at 217.17 48.26 0)
 			(hide yes)
@@
 			)
 		)
-		(property "Stock" "207522"
+		(property "Stock" "464542"
 			(at 217.17 48.26 0)
 			(hide yes)
@@
 			)
 		)
-		(property "Price" "0.005USD"
+		(property "Price" "0.004USD"
 			(at 217.17 48.26 0)
 			(hide yes)
@@
 			)
 		)
-		(property "Part" "0805W8F499JT5E"
+		(property "Part" "0402WGF499JTCE"
 			(at 217.17 48.26 0)
 			(hide yes)
@@
 			)
 		)
-		(property "Power(Watts)" "125mW"
+		(property "Power(Watts)" "62.5mW"
 			(at 217.17 48.26 0)
 			(hide yes)
@@
 			)
 		)
-		(property "Overload Voltage (Max)" "150V"
+		(property "Overload Voltage (Max)" "50V"
 			(at 217.17 48.26 0)
 			(hide yes)
@@
 		)
 		(property "Voltage Rated" "50V"
-			(at 110.998 52.578 0)
+			(at 105.918 52.8462 0)
 			(show_name no)
 			(do_not_autoplace no)
@@
 		)
 		(property "Voltage Rated" "50V"
-			(at 95.758 109.728 0)
+			(at 90.678 109.9962 0)
 			(show_name no)
 			(do_not_autoplace no)
@@
 		)
 		(property "Voltage Rated" "50V"
-			(at 184.658 113.538 0)
+			(at 179.578 113.8062 0)
 			(show_name no)
 			(do_not_autoplace no)
@@
 	)
 	(symbol
-		(lib_id "PCM_JLCPCB-Resistors:0805,49.9Ω")
+		(lib_id "PCM_JLCPCB-Resistors:0402,49.9Ω")
 		(at 34.29 39.37 90)
 		(unit 1)
@@
 			)
 		)
-		(property "Footprint" "PCM_JLCPCB:R_0805"
+		(property "Footprint" "PCM_JLCPCB:R_0402"
 			(at 34.29 41.148 90)
 			(hide yes)
@@
 			)
 		)
-		(property "Datasheet" "https://www.lcsc.com/datasheet/lcsc_datasheet_2206010200_UNI-ROYAL-Uniroyal-Elec-0805W8F499JT5E_C17720.pdf"
+		(property "Datasheet" "https://www.lcsc.com/datasheet/lcsc_datasheet_2205311900_UNI-ROYAL-Uniroyal-Elec-0402WGF499JTCE_C25120.pdf"
 			(at 34.29 39.37 0)
 			(hide yes)
@@
 			)
 		)
-		(property "Description" "125mW Thick Film Resistors 150V ±100ppm/°C ±1% 49.9Ω 0805 Chip Resistor - Surface Mount ROHS"
+		(property "Description" "62.5mW Thick Film Resistors 50V ±100ppm/°C ±1% 49.9Ω 0402 Chip Resistor - Surface Mount ROHS"
 			(at 34.29 39.37 0)
 			(hide yes)
@@
 			)
 		)
-		(property "LCSC" "C17720"
+		(property "LCSC" "C25120"
 			(at 34.29 39.37 0)
 			(hide yes)
@@
 			)
 		)
-		(property "Stock" "207522"
+		(property "Stock" "464542"
 			(at 34.29 39.37 0)
 			(hide yes)
@@
 			)
 		)
-		(property "Price" "0.005USD"
+		(property "Price" "0.004USD"
 			(at 34.29 39.37 0)
 			(hide yes)
@@
 			)
 		)
-		(property "Part" "0805W8F499JT5E"
+		(property "Part" "0402WGF499JTCE"
 			(at 34.29 39.37 0)
 			(hide yes)
@@
 			)
 		)
-		(property "Power(Watts)" "125mW"
+		(property "Power(Watts)" "62.5mW"
 			(at 34.29 39.37 0)
 			(hide yes)
@@
 			)
 		)
-		(property "Overload Voltage (Max)" "150V"
+		(property "Overload Voltage (Max)" "50V"
 			(at 34.29 39.37 0)
 			(hide yes)
@@
 	)
 	(symbol
-		(lib_id "PCM_JLCPCB-Resistors:0805,49.9Ω")
+		(lib_id "PCM_JLCPCB-Resistors:0402,49.9Ω")
 		(at 53.34 55.88 180)
 		(unit 1)
@@
 			)
 		)
-		(property "Footprint" "PCM_JLCPCB:R_0805"
+		(property "Footprint" "PCM_JLCPCB:R_0402"
 			(at 55.118 55.88 90)
 			(hide yes)
@@
 			)
 		)
-		(property "Datasheet" "https://www.lcsc.com/datasheet/lcsc_datasheet_2206010200_UNI-ROYAL-Uniroyal-Elec-0805W8F499JT5E_C17720.pdf"
+		(property "Datasheet" "https://www.lcsc.com/datasheet/lcsc_datasheet_2205311900_UNI-ROYAL-Uniroyal-Elec-0402WGF499JTCE_C25120.pdf"
 			(at 53.34 55.88 0)
 			(hide yes)
@@
 			)
 		)
-		(property "Description" "125mW Thick Film Resistors 150V ±100ppm/°C ±1% 49.9Ω 0805 Chip Resistor - Surface Mount ROHS"
+		(property "Description" "62.5mW Thick Film Resistors 50V ±100ppm/°C ±1% 49.9Ω 0402 Chip Resistor - Surface Mount ROHS"
 			(at 53.34 55.88 0)
 			(hide yes)
@@
 			)
 		)
-		(property "LCSC" "C17720"
+		(property "LCSC" "C25120"
 			(at 53.34 55.88 0)
 			(hide yes)
@@
 			)
 		)
-		(property "Stock" "207522"
+		(property "Stock" "464542"
 			(at 53.34 55.88 0)
 			(hide yes)
@@
 			)
 		)
-		(property "Price" "0.005USD"
+		(property "Price" "0.004USD"
 			(at 53.34 55.88 0)
 			(hide yes)
@@
 			)
 		)
-		(property "Part" "0805W8F499JT5E"
+		(property "Part" "0402WGF499JTCE"
 			(at 53.34 55.88 0)
 			(hide yes)
@@
 			)
 		)
-		(property "Power(Watts)" "125mW"
+		(property "Power(Watts)" "62.5mW"
 			(at 53.34 55.88 0)
 			(hide yes)
@@
 			)
 		)
-		(property "Overload Voltage (Max)" "150V"
+		(property "Overload Voltage (Max)" "50V"
 			(at 53.34 55.88 0)
 			(hide yes)
@@
 		)
 		(property "Voltage Rated" "50V"
-			(at 24.638 36.322 90)
+			(at 24.9062 41.402 0)
 			(show_name no)
 			(do_not_autoplace no)
@@
 		)
 		(property "Voltage Rated" "50V"
-			(at 37.338 104.648 0)
+			(at 32.258 104.9162 0)
 			(show_name no)
 			(do_not_autoplace no)
@@
 		)
 		(property "Voltage Rated" "50V"
-			(at 207.518 45.212 90)
+			(at 207.7862 50.292 0)
 			(show_name no)
 			(do_not_autoplace no)

Commit message: Working on the analog chains
Parts:
- removed R39, R41: 510Ω, PCM_JLCPCB:R_0805, symbol PCM_JLCPCB-Resistors:0805,510Ω
- removed R50, R51: 10Ω, PCM_JLCPCB:R_0603, symbol PCM_JLCPCB-Resistors:0603,10Ω
- added R41, R50: 510Ω, PCM_JLCPCB:R_0402, symbol PCM_JLCPCB-Resistors:0402,510Ω
- added R51, R85: 10Ω, PCM_JLCPCB:R_0402, symbol PCM_JLCPCB-Resistors:0402,10Ω
Connections:
- net at R48.1: now also R51.2, R85.1
- net at U10.1: now also R51.1
- net at R40.2, U17.4 (-): now also R41.1
- net at TP32.1, U17.1, U24.1: now also R41.2
- net at R74.2, TP31.1, U16.1: now also R50.2
- net at R58.2, U13.1: now also R85.2
- net at R38.2, U16.4 (-): now also R50.1
