File: PGA.kicad_sch (KiCad schematic)
At the start: 53 parts, among them Q6 2N7002, Q7 2N7002, Q8 2N7002, Q9 2N7002, U10 74LVC1G3157GW, U13 74LVC1G3157GW, U16 TPH2501-TR, U17 TPH2501-TR, U19 74LVC1G3157GW, U20 74LVC1G3157GW, U21 74LVC1G3157GW, U22 74LVC1G3157GW, U23 74LVC1G3157GW, U24 74LVC1G3157GW

Commit message: AF DAC Some VDDA Placed
Parts:
- renumbered C70 to C81, C78 to C82, C69 to C83, C79 to C84, C73 to C85, C94 to C86, C74 to C87, C80 to C88, C95 to C89, C81 to C90, C71 to C91, C82 to C92, C72 to C93, C83 to C94, Q7 to Q4, Q6 to Q5, Q8 to Q6, Q9 to Q7, R45 to R58, R75 to R59, R38 to R60, R26 to R61, R50 to R62, R74 to R63, R44 to R64, R58 to R65, R85 to R66, R48 to R67, R27 to R68, R51 to R69, R46 to R70, R57 to R71, R49 to R72, R53 to R73, R54 to R74, R29 to R75, R52 to R76, R47 to R77, R40 to R78, R56 to R79, R41 to R80, TP31 to TP10, TP32 to TP11, U19 to U12, U16 to U13, U20 to U14, U13 to U15, U10 to U16, U21 to U17, U22 to U18, U23 to U19, U17 to U20, U24 to U21

Commit message: Fixed schematic errors, all placed
Parts:
- Q4, Q5, Q6, Q7: symbol JLCPCB-Transistors:NMOS,2N7002 -> PCM_JLCPCB-Transistors:NMOS,2N7002K; Attrition Qty 5 -> 4; Category Transistors,MOSFETs -> Triode/MOS Tube/Transistor,MOSFETs; Class Basic Component -> Preferred Component; LCSC C8545 -> C22379475; Manufacturer Changjiang Electronics Tech (CJ) -> hongjiacheng; Part 2N7002 -> 2N7002K; Stock 1078050 -> 82639
Changed lines of the file:
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@@
 	)
 	(symbol
-		(lib_id "JLCPCB-Transistors:NMOS,2N7002")
+		(lib_id "PCM_JLCPCB-Transistors:NMOS,2N7002K")
 		(at 139.7 90.17 0)
 		(unit 1)
@@
 			)
 		)
-		(property "Datasheet" "https://www.lcsc.com/datasheet/lcsc_datasheet_2304140030_Jiangsu-Changjing-Electronics-Technology-Co---Ltd--2N7002_C8545.pdf"
+		(property "Datasheet" "https://wmsc.lcsc.com/wmsc/upload/file/pdf/v2/lcsc/2404091613_hongjiacheng-2N7002K_C22379475.pdf"
 			(at 139.7 90.17 0)
 			(hide yes)
@@
 			)
 		)
-		(property "Description" "60V 115mA 200mW 7.5Ω@10V,500mA 2.5V@250uA 1 N-Channel SOT-23 MOSFETs ROHS"
+		(property "Description" "60V 340mA 350mW 900mΩ@10V,500mA 2.5V@1mA 1PCSNChannel SOT-23 MOSFETs ROHS"
 			(at 139.7 90.17 0)
 			(hide yes)
@@
 			)
 		)
-		(property "LCSC" "C8545"
+		(property "LCSC" "C22379475"
 			(at 139.7 90.17 0)
 			(hide yes)
@@
 			)
 		)
-		(property "Stock" "1078050"
+		(property "Stock" "82639"
 			(at 139.7 90.17 0)
 			(hide yes)
@@
 			)
 		)
-		(property "Attrition Qty" "5"
+		(property "Attrition Qty" "4"
 			(at 139.7 90.17 0)
 			(hide yes)
@@
 			)
 		)
-		(property "Class" "Basic Component"
+		(property "Class" "Preferred Component"
 			(at 139.7 90.17 0)
 			(hide yes)
@@
 			)
 		)
-		(property "Category" "Transistors,MOSFETs"
+		(property "Category" "Triode/MOS Tube/Transistor,MOSFETs"
 			(at 139.7 90.17 0)
 			(hide yes)
@@
 			)
 		)
-		(property "Manufacturer" "Changjiang Electronics Tech (CJ)"
+		(property "Manufacturer" "hongjiacheng"
 			(at 139.7 90.17 0)
 			(hide yes)
@@
 			)
 		)
-		(property "Part" "2N7002"
+		(property "Part" "2N7002K"
 			(at 139.7 90.17 0)
 			(hide yes)
@@
 	)
 	(symbol
-		(lib_id "JLCPCB-Transistors:NMOS,2N7002")
+		(lib_id "PCM_JLCPCB-Transistors:NMOS,2N7002K")
 		(at 198.12 95.25 0)
 		(unit 1)
@@
 			)
 		)
-		(property "Datasheet" "https://www.lcsc.com/datasheet/lcsc_datasheet_2304140030_Jiangsu-Changjing-Electronics-Technology-Co---Ltd--2N7002_C8545.pdf"
+		(property "Datasheet" "https://wmsc.lcsc.com/wmsc/upload/file/pdf/v2/lcsc/2404091613_hongjiacheng-2N7002K_C22379475.pdf"
 			(at 198.12 95.25 0)
 			(hide yes)
@@
 			)
 		)
-		(property "Description" "60V 115mA 200mW 7.5Ω@10V,500mA 2.5V@250uA 1 N-Channel SOT-23 MOSFETs ROHS"
+		(property "Description" "60V 340mA 350mW 900mΩ@10V,500mA 2.5V@1mA 1PCSNChannel SOT-23 MOSFETs ROHS"
 			(at 198.12 95.25 0)
 			(hide yes)
@@
 			)
 		)
-		(property "LCSC" "C8545"
+		(property "LCSC" "C22379475"
 			(at 198.12 95.25 0)
 			(hide yes)
@@
 			)
 		)
-		(property "Stock" "1078050"
+		(property "Stock" "82639"
 			(at 198.12 95.25 0)
 			(hide yes)
@@
 			)
 		)
-		(property "Attrition Qty" "5"
+		(property "Attrition Qty" "4"
 			(at 198.12 95.25 0)
 			(hide yes)
@@
 			)
 		)
-		(property "Class" "Basic Component"
+		(property "Class" "Preferred Component"
 			(at 198.12 95.25 0)
 			(hide yes)
@@
 			)
 		)
-		(property "Category" "Transistors,MOSFETs"
+		(property "Category" "Triode/MOS Tube/Transistor,MOSFETs"
 			(at 198.12 95.25 0)
 			(hide yes)
@@
 			)
 		)
-		(property "Manufacturer" "Changjiang Electronics Tech (CJ)"
+		(property "Manufacturer" "hongjiacheng"
 			(at 198.12 95.25 0)
 			(hide yes)
@@
 			)
 		)
-		(property "Part" "2N7002"
+		(property "Part" "2N7002K"
 			(at 198.12 95.25 0)
 			(hide yes)
@@
 	)
 	(symbol
-		(lib_id "JLCPCB-Transistors:NMOS,2N7002")
+		(lib_id "PCM_JLCPCB-Transistors:NMOS,2N7002K")
 		(at 77.47 86.36 0)
 		(unit 1)
@@
 			)
 		)
-		(property "Datasheet" "https://www.lcsc.com/datasheet/lcsc_datasheet_2304140030_Jiangsu-Changjing-Electronics-Technology-Co---Ltd--2N7002_C8545.pdf"
+		(property "Datasheet" "https://wmsc.lcsc.com/wmsc/upload/file/pdf/v2/lcsc/2404091613_hongjiacheng-2N7002K_C22379475.pdf"
 			(at 77.47 86.36 0)
 			(hide yes)
@@
 			)
 		)
-		(property "Description" "60V 115mA 200mW 7.5Ω@10V,500mA 2.5V@250uA 1 N-Channel SOT-23 MOSFETs ROHS"
+		(property "Description" "60V 340mA 350mW 900mΩ@10V,500mA 2.5V@1mA 1PCSNChannel SOT-23 MOSFETs ROHS"
 			(at 77.47 86.36 0)
 			(hide yes)
@@
 			)
 		)
-		(property "LCSC" "C8545"
+		(property "LCSC" "C22379475"
 			(at 77.47 86.36 0)
 			(hide yes)
@@
 			)
 		)
-		(property "Stock" "1078050"
+		(property "Stock" "82639"
 			(at 77.47 86.36 0)
 			(hide yes)
@@
 			)
 		)
-		(property "Attrition Qty" "5"
+		(property "Attrition Qty" "4"
 			(at 77.47 86.36 0)
 			(hide yes)
@@
 			)
 		)
-		(property "Class" "Basic Component"
+		(property "Class" "Preferred Component"
 			(at 77.47 86.36 0)
 			(hide yes)
@@
 			)
 		)
-		(property "Category" "Transistors,MOSFETs"
+		(property "Category" "Triode/MOS Tube/Transistor,MOSFETs"
 			(at 77.47 86.36 0)
 			(hide yes)
@@
 			)
 		)
-		(property "Manufacturer" "Changjiang Electronics Tech (CJ)"
+		(property "Manufacturer" "hongjiacheng"
 			(at 77.47 86.36 0)
 			(hide yes)
@@
 			)
 		)
-		(property "Part" "2N7002"
+		(property "Part" "2N7002K"
 			(at 77.47 86.36 0)
 			(hide yes)
@@
 	)
 	(symbol
-		(lib_id "JLCPCB-Transistors:NMOS,2N7002")
+		(lib_id "PCM_JLCPCB-Transistors:NMOS,2N7002K")
 		(at 19.05 96.52 0)
 		(unit 1)
@@
 			)
 		)
-		(property "Datasheet" "https://www.lcsc.com/datasheet/lcsc_datasheet_2304140030_Jiangsu-Changjing-Electronics-Technology-Co---Ltd--2N7002_C8545.pdf"
+		(property "Datasheet" "https://wmsc.lcsc.com/wmsc/upload/file/pdf/v2/lcsc/2404091613_hongjiacheng-2N7002K_C22379475.pdf"
 			(at 19.05 96.52 0)
 			(hide yes)
@@
 			)
 		)
-		(property "Description" "60V 115mA 200mW 7.5Ω@10V,500mA 2.5V@250uA 1 N-Channel SOT-23 MOSFETs ROHS"
+		(property "Description" "60V 340mA 350mW 900mΩ@10V,500mA 2.5V@1mA 1PCSNChannel SOT-23 MOSFETs ROHS"
 			(at 19.05 96.52 0)
 			(hide yes)
@@
 			)
 		)
-		(property "LCSC" "C8545"
+		(property "LCSC" "C22379475"
 			(at 19.05 96.52 0)
 			(hide yes)
@@
 			)
 		)
-		(property "Stock" "1078050"
+		(property "Stock" "82639"
 			(at 19.05 96.52 0)
 			(hide yes)
@@
 			)
 		)
-		(property "Attrition Qty" "5"
+		(property "Attrition Qty" "4"
 			(at 19.05 96.52 0)
 			(hide yes)
@@
 			)
 		)
-		(property "Class" "Basic Component"
+		(property "Class" "Preferred Component"
 			(at 19.05 96.52 0)
 			(hide yes)
@@
 			)
 		)
-		(property "Category" "Transistors,MOSFETs"
+		(property "Category" "Triode/MOS Tube/Transistor,MOSFETs"
 			(at 19.05 96.52 0)
 			(hide yes)
@@
 			)
 		)
-		(property "Manufacturer" "Changjiang Electronics Tech (CJ)"
+		(property "Manufacturer" "hongjiacheng"
 			(at 19.05 96.52 0)
 			(hide yes)
@@
 			)
 		)
-		(property "Part" "2N7002"
+		(property "Part" "2N7002K"
 			(at 19.05 96.52 0)
 			(hide yes)

Commit message: Added Prototype Area
Parts:
- TP10, TP11: footprint TestPoint:TestPoint_THTPad_D2.5mm_Drill1.2mm -> RP2040_minimal:TestPoint_THTPad_D2.5mm_Drill1.2mm
Changed lines of the file:
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@@
 			)
 		)
-		(property "Footprint" "TestPoint:TestPoint_THTPad_D2.5mm_Drill1.2mm"
+		(property "Footprint" "RP2040_minimal:TestPoint_THTPad_D2.5mm_Drill1.2mm"
 			(at 240.03 53.34 0)
 			(hide yes)
@@
 			)
 		)
-		(property "Footprint" "TestPoint:TestPoint_THTPad_D2.5mm_Drill1.2mm"
+		(property "Footprint" "RP2040_minimal:TestPoint_THTPad_D2.5mm_Drill1.2mm"
 			(at 57.15 46.99 0)
 			(hide yes)

Commit message: 0 errors 0 warnings
Parts:
- TP10: value U16 -> U13
- TP11: value U17 -> U20
Changed lines of the file:
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@@
 			)
 		)
-		(property "Value" "U17"
+		(property "Value" "U20"
 			(at 241.046 50.292 90)
 			(show_name no)
@@
 			)
 		)
-		(property "Value" "U16"
+		(property "Value" "U13"
 			(at 58.928 39.878 90)
 			(show_name no)
