File: VDDA.kicad_sch (KiCad schematic)
At the start: 45 parts, among them J7 Conn_01x02, Q3 AO3401A, U8 L78M05ABDT-TR

Commit message: VA/2
Connections:
- net VDDA: now also TP5.1
- net at C50.1, C52.1, C54.1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: no longer TP5.1
Changed lines of the file:
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@@
 	)
 	(junction
+		(at 208.28 86.36)
+		(diameter 0)
+		(color 0 0 0 0)
+	)
+	(junction
 		(at 189.23 135.89)
 		(diameter 0)
@@
 	)
 	(junction
-		(at 228.6 100.33)
-		(diameter 0)
-		(color 0 0 0 0)
-	)
-	(junction
 		(at 119.38 100.33)
 		(diameter 0)
@@
 	(wire
 		(pts
-			(xy 228.6 100.33) (xy 248.92 100.33)
-		)
-		(stroke
-			(width 0)
-			(type default)
-		)
-	)
-	(wire
-		(pts
 			(xy 171.45 100.33) (xy 177.8 100.33)
 		)
@@
 	(symbol
 		(lib_id "Connector:TestPoint")
-		(at 248.92 100.33 270)
+		(at 208.28 86.36 270)
 		(unit 1)
 		(body_style 1)
@@
 		(dnp no)
 		(property "Reference" "TP5"
-			(at 255.27 100.33 90)
+			(at 214.63 86.36 90)
 			(hide yes)
 			(show_name no)
@@
 		)
 		(property "Value" "VDDA"
-			(at 251.46 97.79 90)
+			(at 210.82 83.82 90)
 			(show_name no)
 			(do_not_autoplace no)
@@
 		)
 		(property "Footprint" "RP2040_minimal:TestPoint_THTPad_D2.5mm_Drill1.2mm"
-			(at 248.92 105.41 0)
+			(at 208.28 91.44 0)
 			(hide yes)
 			(show_name no)
@@
 		)
 		(property "Datasheet" ""
-			(at 248.92 105.41 0)
+			(at 208.28 91.44 0)
 			(hide yes)
 			(show_name no)
@@
 		)
 		(property "Description" ""
-			(at 248.92 100.33 0)
+			(at 208.28 86.36 0)
 			(hide yes)
 			(show_name no)
@@
 		)
 		(property "JLCPCB #" ""
-			(at 248.92 100.33 0)
+			(at 208.28 86.36 0)
 			(hide yes)
 			(show_name no)
@@
 		)
 		(property "Value" "VDDA"
-			(at 215.138 89.154 90)
+			(at 211.836 90.678 90)
 			(show_name no)
 			(do_not_autoplace no)
