File: VDDA.kicad_sch (KiCad schematic)
At the start: 45 parts, among them J7 Conn_01x02, Q3 AO3401A, U8 L78M05ABDT-TR

Commit message: JLCPCB Order Fixes
Parts:
- R39, R44, R45, R46, R47: footprint PCM_JLCPCB:R_0402 -> PCM_JLCPCB:R_0603; symbol PCM_JLCPCB-Resistors:0402,1Ω -> PCM_JLCPCB-Resistors:0603,1Ω; Class Preferred Component -> Basic Component; LCSC C25086 -> C22936; Overload Voltage (Max) 50V -> 75V; Part 0402WGF100KTCE -> 0603WAF100KT5E; Power(Watts) 62.5mW -> 100mW; Price 0.004USD -> 0.005USD; Stock 305976 -> 632912; Temperature Coefficient ±200ppm/°C -> ±400ppm/°C
Changed lines of the file:
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@@
 	)
 	(symbol
-		(lib_id "PCM_JLCPCB-Resistors:0402,1Ω")
+		(lib_id "PCM_JLCPCB-Resistors:0603,1Ω")
 		(at 105.41 71.12 180)
 		(unit 1)
@@
 			)
 		)
-		(property "Footprint" "PCM_JLCPCB:R_0402"
+		(property "Footprint" "PCM_JLCPCB:R_0603"
 			(at 107.188 71.12 90)
 			(hide yes)
@@
 			)
 		)
-		(property "Datasheet" "https://www.lcsc.com/datasheet/lcsc_datasheet_2205311900_UNI-ROYAL-Uniroyal-Elec-0402WGF100KTCE_C25086.pdf"
+		(property "Datasheet" "https://www.lcsc.com/datasheet/lcsc_datasheet_2206010130_UNI-ROYAL-Uniroyal-Elec-0603WAF100KT5E_C22936.pdf"
 			(at 105.41 71.12 0)
 			(hide yes)
@@
 			)
 		)
-		(property "Description" "62.5mW Thick Film Resistors 50V ±1% ±200ppm/°C 1Ω 0402 Chip Resistor - Surface Mount ROHS"
+		(property "Description" "100mW Thick Film Resistors 75V ±1% ±400ppm/°C 1Ω 0603 Chip Resistor - Surface Mount ROHS"
 			(at 105.41 71.12 0)
 			(hide yes)
@@
 			)
 		)
-		(property "LCSC" "C25086"
+		(property "LCSC" "C22936"
 			(at 105.41 71.12 0)
 			(hide yes)
@@
 			)
 		)
-		(property "Stock" "305976"
+		(property "Stock" "632912"
 			(at 105.41 71.12 0)
 			(hide yes)
@@
 			)
 		)
-		(property "Price" "0.004USD"
+		(property "Price" "0.005USD"
 			(at 105.41 71.12 0)
 			(hide yes)
@@
 			)
 		)
-		(property "Class" "Preferred Component"
+		(property "Class" "Basic Component"
 			(at 105.41 71.12 0)
 			(hide yes)
@@
 			)
 		)
-		(property "Part" "0402WGF100KTCE"
+		(property "Part" "0603WAF100KT5E"
 			(at 105.41 71.12 0)
 			(hide yes)
@@
 			)
 		)
-		(property "Power(Watts)" "62.5mW"
+		(property "Power(Watts)" "100mW"
 			(at 105.41 71.12 0)
 			(hide yes)
@@
 			)
 		)
-		(property "Overload Voltage (Max)" "50V"
+		(property "Overload Voltage (Max)" "75V"
 			(at 105.41 71.12 0)
 			(hide yes)
@@
 			)
 		)
-		(property "Temperature Coefficient" "±200ppm/°C"
+		(property "Temperature Coefficient" "±400ppm/°C"
 			(at 105.41 71.12 0)
 			(hide yes)
@@
 	)
 	(symbol
-		(lib_id "PCM_JLCPCB-Resistors:0402,1Ω")
+		(lib_id "PCM_JLCPCB-Resistors:0603,1Ω")
 		(at 186.69 100.33 90)
 		(unit 1)
@@
 			)
 		)
-		(property "Footprint" "PCM_JLCPCB:R_0402"
+		(property "Footprint" "PCM_JLCPCB:R_0603"
 			(at 186.69 102.108 90)
 			(hide yes)
@@
 			)
 		)
-		(property "Datasheet" "https://www.lcsc.com/datasheet/lcsc_datasheet_2205311900_UNI-ROYAL-Uniroyal-Elec-0402WGF100KTCE_C25086.pdf"
+		(property "Datasheet" "https://www.lcsc.com/datasheet/lcsc_datasheet_2206010130_UNI-ROYAL-Uniroyal-Elec-0603WAF100KT5E_C22936.pdf"
 			(at 186.69 100.33 0)
 			(hide yes)
@@
 			)
 		)
-		(property "Description" "62.5mW Thick Film Resistors 50V ±1% ±200ppm/°C 1Ω 0402 Chip Resistor - Surface Mount ROHS"
+		(property "Description" "100mW Thick Film Resistors 75V ±1% ±400ppm/°C 1Ω 0603 Chip Resistor - Surface Mount ROHS"
 			(at 186.69 100.33 0)
 			(hide yes)
@@
 			)
 		)
-		(property "LCSC" "C25086"
+		(property "LCSC" "C22936"
 			(at 186.69 100.33 0)
 			(hide yes)
@@
 			)
 		)
-		(property "Stock" "305976"
+		(property "Stock" "632912"
 			(at 186.69 100.33 0)
 			(hide yes)
@@
 			)
 		)
-		(property "Price" "0.004USD"
+		(property "Price" "0.005USD"
 			(at 186.69 100.33 0)
 			(hide yes)
@@
 			)
 		)
-		(property "Class" "Preferred Component"
+		(property "Class" "Basic Component"
 			(at 186.69 100.33 0)
 			(hide yes)
@@
 			)
 		)
-		(property "Part" "0402WGF100KTCE"
+		(property "Part" "0603WAF100KT5E"
 			(at 186.69 100.33 0)
 			(hide yes)
@@
 			)
 		)
-		(property "Power(Watts)" "62.5mW"
+		(property "Power(Watts)" "100mW"
 			(at 186.69 100.33 0)
 			(hide yes)
@@
 			)
 		)
-		(property "Overload Voltage (Max)" "50V"
+		(property "Overload Voltage (Max)" "75V"
 			(at 186.69 100.33 0)
 			(hide yes)
@@
 			)
 		)
-		(property "Temperature Coefficient" "±200ppm/°C"
+		(property "Temperature Coefficient" "±400ppm/°C"
 			(at 186.69 100.33 0)
 			(hide yes)
@@
 	)
 	(symbol
-		(lib_id "PCM_JLCPCB-Resistors:0402,1Ω")
+		(lib_id "PCM_JLCPCB-Resistors:0603,1Ω")
 		(at 193.04 138.43 90)
 		(mirror x)
@@
 			)
 		)
-		(property "Footprint" "PCM_JLCPCB:R_0402"
+		(property "Footprint" "PCM_JLCPCB:R_0603"
 			(at 193.04 136.652 90)
 			(hide yes)
@@
 			)
 		)
-		(property "Datasheet" "https://www.lcsc.com/datasheet/lcsc_datasheet_2205311900_UNI-ROYAL-Uniroyal-Elec-0402WGF100KTCE_C25086.pdf"
+		(property "Datasheet" "https://www.lcsc.com/datasheet/lcsc_datasheet_2206010130_UNI-ROYAL-Uniroyal-Elec-0603WAF100KT5E_C22936.pdf"
 			(at 193.04 138.43 0)
 			(hide yes)
@@
 			)
 		)
-		(property "Description" "62.5mW Thick Film Resistors 50V ±1% ±200ppm/°C 1Ω 0402 Chip Resistor - Surface Mount ROHS"
+		(property "Description" "100mW Thick Film Resistors 75V ±1% ±400ppm/°C 1Ω 0603 Chip Resistor - Surface Mount ROHS"
 			(at 193.04 138.43 0)
 			(hide yes)
@@
 			)
 		)
-		(property "LCSC" "C25086"
+		(property "LCSC" "C22936"
 			(at 193.04 138.43 0)
 			(hide yes)
@@
 			)
 		)
-		(property "Stock" "305976"
+		(property "Stock" "632912"
 			(at 193.04 138.43 0)
 			(hide yes)
@@
 			)
 		)
-		(property "Price" "0.004USD"
+		(property "Price" "0.005USD"
 			(at 193.04 138.43 0)
 			(hide yes)
@@
 			)
 		)
-		(property "Class" "Preferred Component"
+		(property "Class" "Basic Component"
 			(at 193.04 138.43 0)
 			(hide yes)
@@
 			)
 		)
-		(property "Part" "0402WGF100KTCE"
+		(property "Part" "0603WAF100KT5E"
 			(at 193.04 138.43 0)
 			(hide yes)
@@
 			)
 		)
-		(property "Power(Watts)" "62.5mW"
+		(property "Power(Watts)" "100mW"
 			(at 193.04 138.43 0)
 			(hide yes)
@@
 			)
 		)
-		(property "Overload Voltage (Max)" "50V"
+		(property "Overload Voltage (Max)" "75V"
 			(at 193.04 138.43 0)
 			(hide yes)
@@
 			)
 		)
-		(property "Temperature Coefficient" "±200ppm/°C"
+		(property "Temperature Coefficient" "±400ppm/°C"
 			(at 193.04 138.43 0)
 			(hide yes)
@@
 	)
 	(symbol
-		(lib_id "PCM_JLCPCB-Resistors:0402,1Ω")
+		(lib_id "PCM_JLCPCB-Resistors:0603,1Ω")
 		(at 193.04 135.89 90)
 		(unit 1)
@@
 			)
 		)
-		(property "Footprint" "PCM_JLCPCB:R_0402"
+		(property "Footprint" "PCM_JLCPCB:R_0603"
 			(at 193.04 137.668 90)
 			(hide yes)
@@
 			)
 		)
-		(property "Datasheet" "https://www.lcsc.com/datasheet/lcsc_datasheet_2205311900_UNI-ROYAL-Uniroyal-Elec-0402WGF100KTCE_C25086.pdf"
+		(property "Datasheet" "https://www.lcsc.com/datasheet/lcsc_datasheet_2206010130_UNI-ROYAL-Uniroyal-Elec-0603WAF100KT5E_C22936.pdf"
 			(at 193.04 135.89 0)
 			(hide yes)
@@
 			)
 		)
-		(property "Description" "62.5mW Thick Film Resistors 50V ±1% ±200ppm/°C 1Ω 0402 Chip Resistor - Surface Mount ROHS"
+		(property "Description" "100mW Thick Film Resistors 75V ±1% ±400ppm/°C 1Ω 0603 Chip Resistor - Surface Mount ROHS"
 			(at 193.04 135.89 0)
 			(hide yes)
@@
 			)
 		)
-		(property "LCSC" "C25086"
+		(property "LCSC" "C22936"
 			(at 193.04 135.89 0)
 			(hide yes)
@@
 			)
 		)
-		(property "Stock" "305976"
+		(property "Stock" "632912"
 			(at 193.04 135.89 0)
 			(hide yes)
@@
 			)
 		)
-		(property "Price" "0.004USD"
+		(property "Price" "0.005USD"
 			(at 193.04 135.89 0)
 			(hide yes)
@@
 			)
 		)
-		(property "Class" "Preferred Component"
+		(property "Class" "Basic Component"
 			(at 193.04 135.89 0)
 			(hide yes)
@@
 			)
 		)
-		(property "Part" "0402WGF100KTCE"
+		(property "Part" "0603WAF100KT5E"
 			(at 193.04 135.89 0)
 			(hide yes)
@@
 			)
 		)
-		(property "Power(Watts)" "62.5mW"
+		(property "Power(Watts)" "100mW"
 			(at 193.04 135.89 0)
 			(hide yes)
@@
 			)
 		)
-		(property "Overload Voltage (Max)" "50V"
+		(property "Overload Voltage (Max)" "75V"
 			(at 193.04 135.89 0)
 			(hide yes)
@@
 			)
 		)
-		(property "Temperature Coefficient" "±200ppm/°C"
+		(property "Temperature Coefficient" "±400ppm/°C"
 			(at 193.04 135.89 0)
 			(hide yes)
@@
 	)
 	(symbol
-		(lib_id "PCM_JLCPCB-Resistors:0402,1Ω")
+		(lib_id "PCM_JLCPCB-Resistors:0603,1Ω")
 		(at 186.69 102.87 90)
 		(mirror x)
@@
 			)
 		)
-		(property "Footprint" "PCM_JLCPCB:R_0402"
+		(property "Footprint" "PCM_JLCPCB:R_0603"
 			(at 186.69 101.092 90)
 			(hide yes)
@@
 			)
 		)
-		(property "Datasheet" "https://www.lcsc.com/datasheet/lcsc_datasheet_2205311900_UNI-ROYAL-Uniroyal-Elec-0402WGF100KTCE_C25086.pdf"
+		(property "Datasheet" "https://www.lcsc.com/datasheet/lcsc_datasheet_2206010130_UNI-ROYAL-Uniroyal-Elec-0603WAF100KT5E_C22936.pdf"
 			(at 186.69 102.87 0)
 			(hide yes)
@@
 			)
 		)
-		(property "Description" "62.5mW Thick Film Resistors 50V ±1% ±200ppm/°C 1Ω 0402 Chip Resistor - Surface Mount ROHS"
+		(property "Description" "100mW Thick Film Resistors 75V ±1% ±400ppm/°C 1Ω 0603 Chip Resistor - Surface Mount ROHS"
 			(at 186.69 102.87 0)
 			(hide yes)
@@
 			)
 		)
-		(property "LCSC" "C25086"
+		(property "LCSC" "C22936"
 			(at 186.69 102.87 0)
 			(hide yes)
@@
 			)
 		)
-		(property "Stock" "305976"
+		(property "Stock" "632912"
 			(at 186.69 102.87 0)
 			(hide yes)
@@
 			)
 		)
-		(property "Price" "0.004USD"
+		(property "Price" "0.005USD"
 			(at 186.69 102.87 0)
 			(hide yes)
@@
 			)
 		)
-		(property "Class" "Preferred Component"
+		(property "Class" "Basic Component"
 			(at 186.69 102.87 0)
 			(hide yes)
@@
 			)
 		)
-		(property "Part" "0402WGF100KTCE"
+		(property "Part" "0603WAF100KT5E"
 			(at 186.69 102.87 0)
 			(hide yes)
@@
 			)
 		)
-		(property "Power(Watts)" "62.5mW"
+		(property "Power(Watts)" "100mW"
 			(at 186.69 102.87 0)
 			(hide yes)
@@
 			)
 		)
-		(property "Overload Voltage (Max)" "50V"
+		(property "Overload Voltage (Max)" "75V"
 			(at 186.69 102.87 0)
 			(hide yes)
@@
 			)
 		)
-		(property "Temperature Coefficient" "±200ppm/°C"
+		(property "Temperature Coefficient" "±400ppm/°C"
 			(at 186.69 102.87 0)
 			(hide yes)
