File: DDC_SDR.kicad_pcb (KiCad board)
At the start: 4 copper layers, 100 x 100 mm, 292 parts, among them J1 Filter, J10 SDR ANT, J11 Filter, J12 Filter, J2 S11, J3 Filter, J4 S21_OUT, J5 AWG_OUT, J6 PMOD, J7 Conn_01x02, J8 OLED, J9 3.5mm_Jack, Q1 2N7002, Q2 2N7002, Q3 AO3401A, Q4 2N7002, Q5 2N7002, Q6 2N7002, Q7 2N7002, Q8 2N7002, Q9 2N7002, SW1 RotaryEncoder_Switch_MP, U1 74LVC1G3157GW, U10 PAM8908, U11 NCP115AMX120TCG, U12 74LVC1G3157GW, U13 TPH2501-TR, U14 74LVC1G3157GW, U15 74LVC1G3157GW, U16 74LVC1G3157GW, U17 74LVC1G3157GW, U18 74LVC1G3157GW, U19 74LVC1G3157GW, U2 TPH2501-TR, U20 TPH2501-TR, U21 74LVC1G3157GW, U22 74LVC1G3157GW, U23 74LVC1G3157GW, U24 74LVC1G3157GW, U3 TPH2501-TR, U4 MS9280, U5 MS9708, U6 74LVC1G3157GW, U7 ICE40UP5K-SG48ITR, U8 L78M05ABDT-TR, U9 CJC4334H, X1 SG-8018CE 30.720000MHz TJHPA

Commit message: Power supplies
Parts:
- moved C82 0.57 mm to (102.2, 90.7)
- moved R59 0.51 mm to (104.5, 92.5)
- moved U12 0.47 mm to (102.1, 93.4)
- moved TP10 0.45 mm to (105.3, 94.8)
- moved C83 0.26 mm to (106.4, 92.5)
Routing:
- net Net-(Q9-D): track 0.00 -> 105.7 mm, vias 0 -> 4
- net Net-(Q6-D): track 0.00 -> 98.3 mm, vias 0 -> 2
- net /ANG_1: track 0.00 -> 92.1 mm, vias 0 -> 2
- net Net-(Q5-D): track 0.00 -> 90.8 mm, vias 0 -> 5
- net Net-(Q7-D): track 0.00 -> 88.5 mm, vias 0 -> 4
- net Net-(Q4-D): track 0.00 -> 86.7 mm, vias 0 -> 4
- net /ANG_0: track 0.00 -> 84.7 mm, vias 0 -> 2
- net /~{REF}: track 0.00 -> 84.1 mm, vias 0 -> 6
- net /ICE_SSN: track 0.00 -> 78.0 mm, vias 0 -> 6
- net /FPGA_INT: track 0.04 -> 76.8 mm, vias 0 -> 3
- net /ANG_2: track 0.00 -> 73.4 mm, vias 0 -> 2
- net Net-(Q8-D): track 0.00 -> 65.1 mm, vias 0 -> 3
- net +4.7V: track 0.00 -> 52.6 mm, vias 0 -> 2
- net /PMOD_2: track 21.3 -> 64.5 mm, vias 1 -> 2
- net Net-(Q3-S): track 0.00 -> 41.5 mm, vias 0 -> 4
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
Commit message: VA/2
Parts:
- removed REF**: Prototype_array, RP2040_minimal:Prototype_array
- moved R57 71.9 mm to (184.5, 146.7), turned to -90 degrees
- moved C78 69.2 mm to (193.5, 131.0), turned to 90 degrees
Connections:
- TP5 pad 1: Net-(JP7-A) -> VDDA
Routing:
- net VA/2: track 0.87 -> 225.8 mm, vias 0 -> 11
- net VDDA: track 24.1 -> 41.2 mm, vias 0 -> 1
- net +4.7V: track 52.6 -> 65.0 mm
- net Net-(e4-B): track 3.58 -> 7.26 mm, vias 0 -> 1
- net Net-(Q2-D): track 0.00 -> 2.57 mm
- net Net-(D4-Pad2): track 0.00 -> 1.51 mm
- net /ANG_2: track 73.4 -> 74.8 mm
- net /ANG_1: track 92.1 -> 92.9 mm

Commit message: 3.3VA
Parts:
- added H1: Prototyping Area, RP2040_minimal:Prototype_array, F.Cu at (150.1, 64.7)
Routing:
- net +3.3VA: track 5.58 -> 132.7 mm, vias 0 -> 3

Commit message: Power Planes started
Parts:
- turned JP7 to 180 degrees
Routing:
- net VDDA: track 41.2 -> 147.1 mm, vias 1 -> 22
- net Net-(Q6-D): track 98.4 -> 99.3 mm
- net +3V3: track 10.8 -> 11.5 mm, vias 0 -> 3
- net Net-(Q7-D): track 88.5 -> 89.1 mm
- net /DB1: track 14.3 -> 13.7 mm
- net +1V2: track 2.42 -> 3.02 mm, vias 0 -> 1
- net /ANG_1: track 92.9 -> 93.4 mm
- net GND: track 0.64 -> 1.12 mm, vias 0 -> 1
- added copper zone on In2.Cu, net +3V3
- added copper zone on In2.Cu, net VDDA
Other:
- board size 100 x 100 mm -> 75 x 75 mm

Commit message: 0 disconnects
Parts:
- moved TP9 12.3 mm to (125.7, 111.2)
- moved C37 1.03 mm to (127.4, 118.4)
- moved C22 0.81 mm to (118.3, 122.9), turned to 0 degrees
- moved C77 0.72 mm to (128.2, 116.7)
- moved C36 0.49 mm to (129.8, 118.4)
- moved C75 0.34 mm to (130.0, 116.1)
- moved C76 0.34 mm to (130.0, 117.0)
Connections:
- C61 pad 2: GNDA -> GND
- C67 pad 2: GNDA -> GND
- R89 pad 2: GNDA -> GND
- U10 pad 10: GNDA -> GND
- U10 pad 15: GNDA -> GND
- U10 pad 17: GNDA -> GND
Routing:
- net GND: track 1.12 -> 246.3 mm, vias 1 -> 118
- net /TX_SDR: track 5.08 -> 122.7 mm, vias 0 -> 2
- net Net-(Q7-D): track 89.1 -> 171.2 mm, vias 4 -> 6
- net +1V2: track 3.02 -> 31.2 mm, vias 1 -> 4
- net +3V3: track 11.5 -> 36.4 mm, vias 3 -> 23
- net /~{REF}: track 84.1 -> 106.6 mm, vias 6 -> 9
- net Net-(Q3-G): track 10.3 -> 28.6 mm, vias 0 -> 2
- net /AF DAC/VAA: track 1.14 -> 16.0 mm, vias 0 -> 4
- net Net-(Q5-D): track 90.6 -> 104.5 mm, vias 5 -> 6
- net VDDA: track 147.1 -> 158.8 mm, vias 22 -> 29
- net Net-(Q6-D): track 99.3 -> 109.4 mm
- net Net-(D8-K): track 0.00 -> 9.67 mm, vias 0 -> 2
- net /FPGA Power/VCC_PLL: track 3.58 -> 12.3 mm, vias 0 -> 2
- net Net-(U10-OUTR): track 9.61 -> 16.1 mm
- net Net-(JP5-A): track 10.2 -> 15.0 mm, vias 0 -> 1
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- added copper zone on In1.Cu, net GND
Other:
- board outline removed
