File: Pico-Dev-iCE.kicad_pcb (KiCad board)
At the start: 4 copper layers, 100 x 100 mm, 292 parts, among them J1 Filter, J10 SDR ANT, J11 Filter, J12 Filter, J2 S11, J3 Filter, J4 S21, J5 AWG_OUT, J6 PMOD, J7 Conn_01x02, J8 OLED, J9 3.5mm_Jack, Q1 2N7002, Q2 2N7002, Q3 AO3401A, Q4 2N7002, Q5 2N7002, Q6 2N7002, Q7 2N7002, Q8 2N7002, Q9 2N7002, SW1 RotaryEncoder_Switch_MP, U1 74LVC1G3157GW, U10 PAM8908, U11 NCP115AMX120TCG, U12 74LVC1G3157GW, U13 TPH2501-TR, U14 74LVC1G3157GW, U15 74LVC1G3157GW, U16 74LVC1G3157GW, U17 74LVC1G3157GW, U18 74LVC1G3157GW, U19 74LVC1G3157GW, U2 TPH2501-TR, U20 TPH2501-TR, U21 74LVC1G3157GW, U22 74LVC1G3157GW, U23 74LVC1G3157GW, U24 74LVC1G3157GW, U3 TPH2501-TR, U4 MS9280, U5 MS9708, U6 74LVC1G3157GW, U7 ICE40UP5K-SG48ITR, U8 L78M05ABDT-TR, U9 CJC4334H, X1 SG-8018CE 30.720000MHz TJHPA

Commit message: JLCPCB Order Fixes
Parts:
- removed J1, J11, J12, J3: Filter, Connector_PinSocket_2.54mm:PinSocket_1x04_P2.54mm_Vertical
- added Je3: Filter, Connector_PinHeader_2.54mm:PinHeader_1x04_P2.54mm_Vertical, F.Cu at (149.4, 146.9)
- added Je4: Filter, Connector_PinHeader_2.54mm:PinHeader_1x04_P2.54mm_Vertical, F.Cu at (159.2, 135.6)
- added Je5: Filter, Connector_PinHeader_2.54mm:PinHeader_1x04_P2.54mm_Vertical, F.Cu at (110.1, 79.3)
- added Je6: Filter, Connector_PinHeader_2.54mm:PinHeader_1x04_P2.54mm_Vertical, F.Cu at (102.0, 75.1)
- R39, R44, R45, R46, R47: footprint PCM_JLCPCB:R_0402 -> PCM_JLCPCB:R_0603
- moved R46 0.59 mm to (190.3, 78.2)
- moved R44 0.59 mm to (172.6, 96.2)
- moved R39 0.41 mm to (188.9, 100.8)
- moved R47 0.39 mm to (190.3, 79.5)
- moved R45 0.32 mm to (172.6, 97.6)
- moved C39 0.15 mm to (189.3, 99.2)
Routing:
- net Net-(FB5-Pad1): track 4.21 -> 5.11 mm
- net Net-(FB4-Pad1): track 2.97 -> 3.53 mm
- net GND: vias 165 -> 173
