File: Pico-Dev-iCE.kicad_sch (KiCad schematic)
At the start: 108 parts, among them J1 Filter, J2 S11, J3 Filter, J4 S21, J5 AWG_OUT, J6 PMOD, Q1 2N7002, Q2 2N7002, U1 74LVC1G3157GW, U2 TPH2501-TR, U3 TPH2501-TR, U4 MS9280, U5 MS9708, U6 74LVC1G3157GW, U7 ICE40UP5K-SG48ITR

Commit message: JLCPCB Order Fixes
Parts:
- removed J1, J3: Filter, Connector_PinSocket_2.54mm:PinSocket_1x04_P2.54mm_Vertical, symbol Connector:Conn_01x04_Socket
- removed R28: 10kΩ, PCM_JLCPCB:R_0402, symbol PCM_JLCPCB-Resistors:0402,49.9Ω
- added Je3, Je4: Filter, Connector_PinHeader_2.54mm:PinHeader_1x04_P2.54mm_Vertical, symbol Connector:Conn_01x04_Socket
- added R28: 10kΩ, PCM_JLCPCB:R_0402, symbol PCM_JLCPCB-Resistors:0402,10kΩ
- J2, J4: LCSC (none) -> C52766461
- J5: now not fitted
- J6: LCSC (none) -> C52148815
Connections:
- net +3V3: now also R28.1
- net GND: now also Je3.3 (Pin_3), Je4.2 (Pin_2), Je4.3 (Pin_3)
- net at C19.1: now also Je4.4 (Pin_4)
- net at C5.1: now also Je3.4 (Pin_4)
- net at C2.2: now also Je3.1 (Pin_1)
- net at JP2.2 (B), S1.2 (B): now also R28.2
- net at C9.2: now also Je4.1 (Pin_1)
