File: _restore_backup_2026-07-20T08-11-43-082/FPGA_Power.kicad_sch (KiCad schematic)
At the start: 13 parts, among them U5 NCP115AMX120TCG, U9 ICE40UP5K-SG48ITR

Commit message: Much Schematic Progress
Parts:
- removed C33, C39, C51, C54: 100nF, PCM_JLCPCB:C_0402, symbol PCM_JLCPCB-Capacitors:0402,100nF,(2)
- removed C56, C60, C61, C62: 4.7uF, PCM_JLCPCB:C_0402, symbol PCM_JLCPCB-Capacitors:0402,4.7uF
- added C52, C60, C63, C8: 4.7u, Capacitor_SMD:C_0402_1005Metric, symbol UPduino_v3.0:Device_C
- added C54, C56, C61, C62: 0.1u, Capacitor_SMD:C_0402_1005Metric, symbol UPduino_v3.0:Device_C
Connections:
- net +1.2V_CORE: now also C56.1, C62.1
- net +1V2: now also C52.1
- net +3V3: now also C54.1, C8.1
- net GND: now also C52.2, C54.2, C56.2, C60.2, C61.2, C62.2, C63.2, C8.2
- net VCC_PLL: now also C61.1, C63.1
- net at D5.1 (K), U9.24 (VPP_2V5): now also C60.1
