File: _restore_backup_2026-07-20T12-34-04-072/filter_playground.kicad_sch (KiCad schematic)
At the start: 18 parts, among them J1 Filter, J11 SDR ANT, J2 Filter, Q4 2N7002, Q5 2N7002, U11 74LVC1G3157GW, U14 74LVC1G3157GW, U18 74LVC1G3157GW

Commit message: Much Schematic Progress
Parts:
- removed C6: 100nF, PCM_JLCPCB:C_0402, symbol PCM_JLCPCB-Capacitors:0402,100nF,(2)
Connections:
- net at TR1.8 (RD-): now also U11.4
- net +3.3VA renamed +3V3
- net ~{T}/R renamed ~{TX}
