File: _restore_backup_2026-07-27T15-21-18-564/DDC_SDR.kicad_pcb (KiCad board)
At the start: 4 copper layers, 100 x 100 mm, 292 parts, among them J1 Filter, J10 SDR ANT, J11 Filter, J12 Filter, J2 S11, J3 Filter, J4 S21, J5 AWG_OUT, J6 PMOD, J7 Conn_01x02, J8 OLED, J9 3.5mm_Jack, Q1 2N7002, Q2 2N7002, Q3 AO3401A, Q4 2N7002, Q5 2N7002, Q6 2N7002, Q7 2N7002, Q8 2N7002, Q9 2N7002, SW1 RotaryEncoder_Switch_MP, U1 74LVC1G3157GW, U10 PAM8908, U11 NCP115AMX120TCG, U12 74LVC1G3157GW, U13 TPH2501-TR, U14 74LVC1G3157GW, U15 74LVC1G3157GW, U16 74LVC1G3157GW, U17 74LVC1G3157GW, U18 74LVC1G3157GW, U19 74LVC1G3157GW, U2 TPH2501-TR, U20 TPH2501-TR, U21 74LVC1G3157GW, U22 74LVC1G3157GW, U23 74LVC1G3157GW, U24 74LVC1G3157GW, U3 TPH2501-TR, U4 MS9280, U5 MS9708, U6 74LVC1G3157GW, U7 ICE40UP5K-SG48ITR, U8 L78M05ABDT-TR, U9 CJC4334H, X1 SG-8018CE 30.720000MHz TJHPA

Commit message: Added ground planes
Routing:
- net GND: track 288.7 -> 253.1 mm, vias 157 -> 118
- net +3.3VA: track 134.3 -> 133.3 mm
- net /SPI0_RX: track 69.2 -> 68.6 mm
- net /~{ICE_RST}: track 39.3 -> 38.8 mm
- removed copper zone on B.Cu, net GND
- removed copper zone on F.Cu, net GND
