File: Filter_Board/Filter_Board.kicad_pcb (KiCad board)
At the start: 2 copper layers, 33 x 33 mm, 20 parts, among them J1 PCB Connector, J14 IN, J15 OUT

Commit message: Added board label to filter playground
Other:
- board text added: "Filter Playground v 0.1"
- board text added: "Walla Walla University"
