File: _restore_backup_2026-07-29T09-59-15-652/FPGA_Power.kicad_sch (KiCad schematic)
At the start: 13 parts, among them U11 NCP115AMX120TCG, U7 ICE40UP5K-SG48ITR

Commit message: Getting ready to submit to JLCPCB.
Parts:
- U7: JLCPCB Rotation Offset (none) -> -90
Changed lines of the file:
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@@
 			)
 		)
-		(property "JLCPCB Rotation Offset" ""
+		(property "JLCPCB Rotation Offset" "-90"
 			(at 212.09 106.68 90)
 			(hide yes)
