File: _restore_backup_2026-07-29T09-59-15-652/Pico-Dev-iCE.kicad_pcb (KiCad board)
At the start: 4 copper layers, 100 x 100 mm, 294 parts, among them J10 SDR ANT, J11 Conn_01x20_Socket, J12 Conn_01x20_Socket, J2 S11, J4 S21, J5 AWG_OUT, J6 PMOD, J7 Conn_01x02, J8 OLED, J9 3.5mm_Jack, Q1 2N7002, Q2 2N7002, Q3 AO3401A, Q4 2N7002, Q5 2N7002, Q6 2N7002, Q7 2N7002, Q8 2N7002, Q9 2N7002, SW1 RotaryEncoder_Switch_MP, U1 74LVC1G3157GW, U10 PAM8908, U11 NCP115AMX120TCG, U12 74LVC1G3157GW, U13 TPH2501-TR, U14 74LVC1G3157GW, U15 74LVC1G3157GW, U16 74LVC1G3157GW, U17 74LVC1G3157GW, U18 74LVC1G3157GW, U19 74LVC1G3157GW, U2 TPH2501-TR, U20 TPH2501-TR, U21 74LVC1G3157GW, U22 74LVC1G3157GW, U23 74LVC1G3157GW, U24 74LVC1G3157GW, U3 TPH2501-TR, U4 MS9280, U5 MS9708, U6 74LVC1G3157GW, U7 ICE40UP5K-SG48ITR, U8 L78M05ABDT-TR, U9 CJC4334H, X1 SG-8018CE 30.720000MHz TJHPA

Commit message: Getting ready to submit to JLCPCB.
Parts:
- moved R28 152.0 mm to (0.93, 0.42)
- moved R33 0.28 mm to (185.8, 93.1)
- moved Q3 0.19 mm to (175.7, 94.6)
- moved D7 0.15 mm to (181.1, 94.5)
- moved R42 0.15 mm to (171.8, 106.3)
- moved C46 0.10 mm to (171.9, 104.7)
- moved R38 0.08 mm to (175.8, 97.7)
Connections:
- J11 pad 13: GND -> Net-(J11-Pin_13)
- J11 pad 18: GND -> Net-(J11-Pin_18)
- J12 pad 23: GND -> Net-(J11-Pin_18)
- J12 pad 28: GND -> Net-(J11-Pin_13)
- J12 pad 31: /REF -> /GP27
- J12 pad 32: /GP27 -> /REF
- J12 pad 33: GND -> unconnected-(J12-Pin_8-Pad33)
Routing:
- net /RX_DATA: track 29.4 -> 29.9 mm
