File: _restore_backup_2026-07-29T09-59-15-652/filter_playground.kicad_sch (KiCad schematic)
At the start: 32 parts, among them J10 SDR ANT, Q8 2N7002, Q9 2N7002, U22 74LVC1G3157GW, U23 74LVC1G3157GW, U24 74LVC1G3157GW

Commit message: Getting ready to submit to JLCPCB.
Parts:
- TR4: JLCPCB Rotation Offset (none) -> 180
Changed lines of the file:
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@@
 			)
 		)
-		(property "JLCPCB Rotation Offset" ""
-			(at 115.57 82.55 90)
-			(hide yes)
-			(show_name no)
-			(do_not_autoplace no)
-			(effects
-				(font
-					(size 1.27 1.27)
-				)
-			)
-		)
 		(pin "4"
 		)
@@
 			)
 		)
-		(property "JLCPCB Rotation Offset" ""
-			(at 29.21 72.39 0)
-			(hide yes)
-			(show_name no)
-			(do_not_autoplace no)
-			(effects
-				(font
-					(size 1.27 1.27)
-				)
-			)
-		)
 		(pin "1"
 		)
@@
 			)
 		)
-		(property "JLCPCB Rotation Offset" ""
+		(property "JLCPCB Rotation Offset" "180"
 			(at 59.69 80.01 0)
 			(hide yes)
@@
 			(hide yes)
 			(show_name no)
-			(do_not_autoplace no)
-			(effects
-				(font
-					(size 1.27 1.27)
-				)
-			)
-		)
-		(property "JLCPCB Rotation Offset" ""
-			(at 115.57 62.23 90)
-			(hide yes)
-			(show_name no)
