File: Hardware/Pico-Dev-iCE.kicad_sch (KiCad schematic)
At the start: 110 parts, among them J11 Conn_01x20_Socket, J12 Conn_01x20_Socket, J2 S11, J4 S21, J5 AWG_OUT, J6 PMOD, Q1 2N7002, Q2 2N7002, U1 74LVC1G3157GW, U2 TPH2501-TR, U3 TPH2501-TR, U4 MS9280, U5 MS9708, U6 74LVC1G3157GW, U7 ICE40UP5K-SG48ITR

Commit message: fixed U4 ad SMA footprints
Parts:
- J2, J4: footprint Connector_Coaxial:SMA_Amphenol_132289_EdgeMount -> Connector_Coaxial:SMA_Samtec_SMA-J-P-H-ST-EM1_EdgeMount
- U4: footprint Package_SO:TSSOP-28-1EP_4.4x9.7mm_P0.65mm_EP3.4x9.7mm_Mask3.1x4.05mm_ThermalVias -> Package_SO:SSOP-28_5.3x10.2mm_P0.65mm
Connections:
- net 30: now reaches A1.30 (RUN)
- net 30: now also J12.30 (Pin_11)
- net 35: now reaches A1.35 (ADC_VREF)
- net 35: now also J12.35 (Pin_6)
- net 37: now reaches A1.37 (3V3_EN)
- net 37: now also J12.37 (Pin_4)
- no-connect marks 29 -> 23
Changed lines of the file:
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@@
 	)
 	(no_connect
-		(at 341.63 78.74)
-	)
-	(no_connect
 		(at 43.18 97.79)
 	)
@@
 	)
 	(no_connect
-		(at 330.2 205.74)
-	)
-	(no_connect
 		(at 48.26 213.36)
 	)
@@
 	)
 	(no_connect
-		(at 387.35 50.8)
-	)
-	(no_connect
 		(at 48.26 233.68)
 	)
@@
 	)
 	(no_connect
-		(at 330.2 193.04)
-	)
-	(no_connect
 		(at 35.56 77.47)
 	)
 	(no_connect
-		(at 330.2 187.96)
-	)
-	(no_connect
 		(at 45.72 77.47)
 	)
 	(no_connect
-		(at 387.35 48.26)
-	)
-	(no_connect
 		(at 40.64 213.36)
 	)
@@
 		)
 	)
+	(label "30"
+		(at 387.35 48.26 0)
+		(effects
+			(font
+				(size 1.27 1.27)
+			)
+			(justify left bottom)
+		)
+	)
 	(label "D0"
 		(at 264.16 54.61 0)
@@
 		)
 	)
+	(label "35"
+		(at 330.2 193.04 0)
+		(effects
+			(font
+				(size 1.27 1.27)
+			)
+			(justify left bottom)
+		)
+	)
 	(label "PMOD_3"
 		(at 233.68 91.44 180)
@@
 		)
 	)
+	(label "37"
+		(at 330.2 187.96 0)
+		(effects
+			(font
+				(size 1.27 1.27)
+			)
+			(justify left bottom)
+		)
+	)
 	(label "D3"
 		(at 144.78 63.5 0)
@@
 		)
 	)
+	(label "30"
+		(at 330.2 205.74 0)
+		(effects
+			(font
+				(size 1.27 1.27)
+			)
+			(justify left bottom)
+		)
+	)
 	(label "RX_OUT"
 		(at 20.32 31.75 0)
@@
 		)
 	)
+	(label "35"
+		(at 341.63 78.74 180)
+		(effects
+			(font
+				(size 1.27 1.27)
+			)
+			(justify right bottom)
+		)
+	)
 	(label "REF"
 		(at 330.2 203.2 0)
@@
 		)
 	)
+	(label "37"
+		(at 387.35 50.8 0)
+		(effects
+			(font
+				(size 1.27 1.27)
+			)
+			(justify left bottom)
+		)
+	)
 	(label "ANG_2"
 		(at 364.49 157.48 180)
@@
 			)
 		)
-		(property "Footprint" "Package_SO:TSSOP-28-1EP_4.4x9.7mm_P0.65mm_EP3.4x9.7mm_Mask3.1x4.05mm_ThermalVias"
+		(property "Footprint" "Package_SO:SSOP-28_5.3x10.2mm_P0.65mm"
 			(at 127 58.42 0)
 			(hide yes)
@@
 			)
 		)
-		(property "Footprint" "Connector_Coaxial:SMA_Amphenol_132289_EdgeMount"
+		(property "Footprint" "Connector_Coaxial:SMA_Samtec_SMA-J-P-H-ST-EM1_EdgeMount"
 			(at 48.26 111.76 0)
 			(hide yes)
@@
 			)
 		)
-		(property "Footprint" "Connector_Coaxial:SMA_Amphenol_132289_EdgeMount"
+		(property "Footprint" "Connector_Coaxial:SMA_Samtec_SMA-J-P-H-ST-EM1_EdgeMount"
 			(at 102.87 219.71 0)
 			(hide yes)
